File: Hardware/LEDCircuit/LEDCircuit.kicad_pcb (KiCad board)
At the start: 2 copper layers, 17 x 20 mm, 6 parts, among them J1 Conn_01x02, SW1 SW_Push

Commit message: fix front copper zone
Routing:
- net +3V3: track 9.85 -> 0.00 mm
- added copper zone on F.Cu, net +3V3
- removed copper zone on F.Cu, net (none)
Changed lines of the file:
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@@
-	)
-	(segment
-		(start 144.4 99.2)
-		(end 143.58 100.02)
-		(width 0.25)
-		(layer "F.Cu")
-		(net 3)
-	)
-	(segment
-		(start 143.58 100.02)
-		(end 141.77 100.02)
-		(width 0.25)
-		(layer "F.Cu")
-		(net 3)
-	)
-	(segment
-		(start 145.2 97.4)
-		(end 144.4 98.2)
-		(width 0.25)
-		(layer "F.Cu")
-		(net 3)
-	)
-	(segment
-		(start 147 97.4)
-		(end 145.2 97.4)
-		(width 0.25)
-		(layer "F.Cu")
-		(net 3)
-	)
-	(segment
-		(start 144.4 98.2)
-		(end 144.4 99.2)
-		(width 0.25)
-		(layer "F.Cu")
-		(net 3)
-	)
-	(segment
-		(start 148 96.4)
-		(end 147 97.4)
-		(width 0.25)
-		(layer "F.Cu")
-		(net 3)
-	)
-	(segment
-		(start 148 94.865)
-		(end 148 96.4)
-		(width 0.25)
-		(layer "F.Cu")
-		(net 3)
 	)
 	(segment
@@
 	)
 	(zone
-		(net 0)
-		(net_name "")
+		(net 3)
+		(net_name "+3V3")
 		(layer "F.Cu")
 		(hatch edge 0.5)
