File: Hardware/yjayara2_Horns_v1.0/yjayara2_Horns_v1.0.kicad_sch (KiCad schematic)
At the start: 0 parts

Commit message: Complete Horn Breakout Board PCB layout, passes DRC
Parts:
- added C1, C3, C4, C5, C6, C7: C, Capacitor_SMD:C_0805_2012Metric, symbol device:C
- added C2: C_Polarized, Capacitor_THT:CP_Radial_D5.0mm_P2.00mm, symbol Device:C_Polarized
- added D1: D, Diode_SMD:D_SMA, symbol Device:D
- added D2: LED, LED_THT:LED_D5.0mm, symbol Device:LED
- added F1: Fuse, Fuse:Fuseholder_Cylinder-5x20mm_Bulgin_FX0456_Vertical_Closed, symbol Device:Fuse
- added J1: Conn_01x03, Connector_PinHeader_2.54mm:PinHeader_1x03_P2.54mm_Vertical, symbol Connector_Generic:Conn_01x03
- added J2, J3, J4: Conn_01x02, Connector_PinHeader_2.54mm:PinHeader_1x02_P2.54mm_Vertical, symbol Connector_Generic:Conn_01x02
- added Q1: Q_NMOS, yjayara2_footprints:TO-252-2_GDS, symbol Device:Q_NMOS
- added R1, R2: R, Resistor_SMD:R_0805_2012Metric, symbol device:R
- added SW1: SW_Push, Button_Switch_THT:SW_PUSH_6mm, symbol Switch:SW_Push
- added TP1: TestPoint, TestPoint:TestPoint_Pad_D1.0mm, symbol Connector:TestPoint
Connections:
- new net: F1.2, J3.1 (Pin_1)
- new net: D2.2 (A), R2.2
- new net +24V: C1.1, C3.1, C4.1, C5.1, C6.1, C7.1, D1.2 (A), F1.1, J1.2 (Pin_2)
- new net GND: C1.2, C2.2, C3.2, C4.2, C5.2, C6.2, C7.2, D2.1 (K), J1.1 (Pin_1), J1.3 (Pin_3), J2.1 (Pin_1), Q1.S, SW1.1
- new net HORN_CTL: C2.1, J2.2 (Pin_2), Q1.G, R1.1, R1.2, SW1.2, TP1.1
- new net HORN_IN: D1.1 (K), J4.2 (Pin_2), Q1.D, R2.1
- new net HORN_MID: J3.2 (Pin_2), J4.1 (Pin_1)
Other:
- title: Template -> Horn Breakout Board
