File: Hardware/Horns_Board V1.0/gwharty2_Horns.kicad_pcb (KiCad board)
At the start: 2 copper layers, 0 parts

Commit message: updated horns PCB (passed DRC)
Parts:
- added C1: .1u, Capacitor_SMD:C_0603_1608Metric_Pad1.08x0.95mm_HandSolder, F.Cu at (152.6, 106.7)
- added C2: .1u, Capacitor_SMD:C_0603_1608Metric_Pad1.08x0.95mm_HandSolder, F.Cu at (160.9, 91.5)
- added C3: .1u, Capacitor_SMD:C_0603_1608Metric_Pad1.08x0.95mm_HandSolder, F.Cu at (160.9, 93.2)
- added C4: .1u, Capacitor_SMD:C_0603_1608Metric_Pad1.08x0.95mm_HandSolder, F.Cu at (161.0, 95.0)
- added C5: 1u, Capacitor_SMD:C_0603_1608Metric_Pad1.08x0.95mm_HandSolder, F.Cu at (160.9, 96.8)
- added C6: 1u, Capacitor_SMD:C_0603_1608Metric_Pad1.08x0.95mm_HandSolder, F.Cu at (161.0, 98.7)
- added C7: 10u, Capacitor_SMD:C_0603_1608Metric_Pad1.08x0.95mm_HandSolder, F.Cu at (161.1, 100.5)
- added C8: 10u, Capacitor_SMD:C_0603_1608Metric_Pad1.08x0.95mm_HandSolder, F.Cu at (161.0, 102.4)
- added C9: 100u, Capacitor_SMD:C_Elec_3x5.4, F.Cu at (159.4, 106.3)
- added D1: S2JTR, Diode_SMD:D_SMB, F.Cu at (138.3, 97.4)
- added F1: 2A, Fuse:Fuse_0603_1608Metric_Pad1.05x0.95mm_HandSolder, F.Cu at (150.7, 92.3)
- added J1: Conn_01x03, Connector_Molex:Molex_KK-254_AE-6410-03A_1x03_P2.54mm_Vertical, F.Cu at (138.1, 103.8)
- added J2: Conn_01x02, Connector_Molex:Molex_KK-254_AE-6410-02A_1x02_P2.54mm_Vertical, F.Cu at (153.9, 89.3)
- added J3: Conn_01x02, Connector_Molex:Molex_KK-254_AE-6410-02A_1x02_P2.54mm_Vertical, F.Cu at (138.6, 90.9)
- added J4: Conn_01x02, Connector_Molex:Molex_KK-254_AE-6410-02A_1x02_P2.54mm_Vertical, F.Cu at (145.2, 90.8)
- added Q1: STD7NK40Z, Package_TO_SOT_SMD:TO-252-2, F.Cu at (151.6, 99.5)
- added R1: 1k, Resistor_SMD:R_0603_1608Metric_Pad0.98x0.95mm_HandSolder, F.Cu at (148.6, 106.7)
- added REF**: MountingHole_3.2mm_M3, MountingHole:MountingHole_3.2mm_M3, F.Cu at (132.8, 89.5)
- added REF**: MountingHole_3.2mm_M3, MountingHole:MountingHole_3.2mm_M3, F.Cu at (132.8, 108.0)
- added REF**: MountingHole_3.2mm_M3, MountingHole:MountingHole_3.2mm_M3, F.Cu at (167.3, 108.0)
- added REF**: MountingHole_3.2mm_M3, MountingHole:MountingHole_3.2mm_M3, F.Cu at (167.3, 89.5)
Routing:
- net /HRN_CNTRL: track 0.00 -> 40.5 mm
- net GND: track 0.00 -> 14.8 mm, vias 0 -> 9
- net Net-(D1-K): track 0.00 -> 12.6 mm
- net Net-(Q1-D): track 0.00 -> 8.83 mm
- net +24V: track 0.00 -> 6.47 mm
- net Net-(J3-Pin_2): track 0.00 -> 4.09 mm
- net /HRN_IN: track 0.00 -> 3.26 mm
- net Net-(C1-Pad1): track 0.00 -> 2.20 mm
- added copper zone on F.Cu, net +24V
- added copper zone on B.Cu, net GND
Other:
- board outline added: 43.7 x 28.1 mm

Commit message: LED_proj, Horns, FW#1 finished
Routing:
- net /HRN_CNTRL: track 40.5 -> 39.7 mm
- net Net-(D1-K): track 12.6 -> 12.0 mm
Changed lines of the file:
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@@
 	)
 	(segment
-		(start 154.8 106.7)
-		(end 153.425 106.7)
-		(width 0.25)
-		(layer "F.Cu")
-		(net 2)
-	)
-	(segment
-		(start 157.84 103.56)
-		(end 157.7 103.7)
+		(start 157.84 103.21)
+		(end 157.35 103.7)
+		(width 0.25)
+		(layer "F.Cu")
+		(net 2)
+	)
+	(segment
+		(start 154.8 106.3)
+		(end 154.4 106.7)
+		(width 0.25)
+		(layer "F.Cu")
+		(net 2)
+	)
+	(segment
+		(start 147 95.1)
+		(end 146.4 95.1)
 		(width 0.25)
 		(layer "F.Cu")
@@
 	)
 	(segment
+		(start 158.25 89.3)
+		(end 158.65 89.7)
+		(width 0.25)
+		(layer "F.Cu")
+		(net 2)
+	)
+	(segment
+		(start 158.65 89.7)
+		(end 158.65 92.8)
+		(width 0.25)
+		(layer "F.Cu")
+		(net 2)
+	)
+	(segment
+		(start 157.84 93.61)
+		(end 157.84 103.21)
+		(width 0.25)
+		(layer "F.Cu")
+		(net 2)
+	)
+	(segment
+		(start 156.44 89.3)
+		(end 158.25 89.3)
+		(width 0.25)
+		(layer "F.Cu")
+		(net 2)
+	)
+	(segment
+		(start 157.35 103.7)
+		(end 155.8 103.7)
+		(width 0.25)
+		(layer "F.Cu")
+		(net 2)
+	)
+	(segment
 		(start 154.8 104.7)
-		(end 154.8 106.7)
-		(width 0.25)
-		(layer "F.Cu")
-		(net 2)
-	)
-	(segment
-		(start 147.4 95.2)
-		(end 147.3 95.1)
+		(end 154.8 106.3)
+		(width 0.25)
+		(layer "F.Cu")
+		(net 2)
+	)
+	(segment
+		(start 146.4 95.1)
+		(end 145.6 95.9)
 		(width 0.25)
 		(layer "F.Cu")
@@
 	)
 	(segment
-		(start 147.4 97.22)
-		(end 147.4 95.2)
-		(width 0.25)
-		(layer "F.Cu")
-		(net 2)
-	)
-	(segment
-		(start 146.4 95.1)
-		(end 145.6 95.9)
-		(width 0.25)
-		(layer "F.Cu")
-		(net 2)
-	)
-	(segment
-		(start 158.65 89.3)
-		(end 156.44 89.3)
-		(width 0.25)
-		(layer "F.Cu")
-		(net 2)
-	)
-	(segment
 		(start 146 106.7)
 		(end 147.675 106.7)
@@
 	)
 	(segment
-		(start 157.84 93.61)
-		(end 157.84 103.56)
-		(width 0.25)
-		(layer "F.Cu")
-		(net 2)
-	)
-	(segment
-		(start 147.3 95.1)
-		(end 146.4 95.1)
-		(width 0.25)
-		(layer "F.Cu")
-		(net 2)
-	)
-	(segment
-		(start 158.65 92.8)
-		(end 158.65 89.3)
-		(width 0.25)
-		(layer "F.Cu")
-		(net 2)
-	)
-	(segment
-		(start 157.7 103.7)
-		(end 155.8 103.7)
+		(start 155.8 103.7)
+		(end 154.8 104.7)
 		(width 0.25)
 		(layer "F.Cu")
@@
 	)
 	(segment
-		(start 155.8 103.7)
-		(end 154.8 104.7)
+		(start 147.4 97.22)
+		(end 147.4 95.5)
+		(width 0.25)
+		(layer "F.Cu")
+		(net 2)
+	)
+	(segment
+		(start 154.4 106.7)
+		(end 153.425 106.7)
+		(width 0.25)
+		(layer "F.Cu")
+		(net 2)
+	)
+	(segment
+		(start 147.4 95.5)
+		(end 147 95.1)
 		(width 0.25)
 		(layer "F.Cu")
@@
 	)
 	(segment
-		(start 138.56 90.9)
-		(end 136.6 90.9)
+		(start 136.5 91.4)
+		(end 136.5 92.2)
+		(width 0.25)
+		(layer "F.Cu")
+		(net 7)
+	)
+	(segment
+		(start 133.4 96.8)
+		(end 134 97.4)
 		(width 0.25)
 		(layer "F.Cu")
@@
 	(segment
 		(start 133.4 95.3)
-		(end 133.4 97.4)
-		(width 0.25)
-		(layer "F.Cu")
-		(net 7)
-	)
-	(segment
-		(start 133.4 97.4)
-		(end 136.2 97.4)
+		(end 133.4 96.8)
 		(width 0.25)
 		(layer "F.Cu")
@@
 	)
 	(segment
-		(start 136.5 91)
-		(end 136.5 92.2)
-		(width 0.25)
-		(layer "F.Cu")
-		(net 7)
-	)
-	(segment
-		(start 136.6 90.9)
-		(end 136.5 91)
-		(width 0.25)
-		(layer "F.Cu")
+		(start 137 90.9)
+		(end 136.5 91.4)
+		(width 0.25)
+		(layer "F.Cu")
+		(net 7)
+	)
+	(segment
+		(start 134 97.4)
+		(end 136.2 97.4)
+		(width 0.25)
+		(layer "F.Cu")
+		(net 7)
+	)
+	(segment
+		(start 138.56 90.9)
+		(end 137 90.9)
+		(width 0.25)
+		(layer "F.Cu")
