File: Hardware/Dev/Template_v0.0/Template_v0.0.kicad_pcb (KiCad board)
At the start: 2 copper layers, 0 parts

Commit message: First hardware project done
Parts:
- added D1: LED_RED, layout:LED_0603_Symbol_on_F.SilkS, F.Cu at (130.3, 111.4)
- added J1: Conn_01x02, Connector_Molex:Molex_KK-254_AE-6410-02A_1x02_P2.54mm_Vertical, F.Cu at (130.8, 117.0)
- added R1: 105, Resistor_SMD:R_0603_1608Metric_Pad0.98x0.95mm_HandSolder, F.Cu at (134.0, 111.3)
- added REF**: MountingHole_3.2mm_M3, MountingHole:MountingHole_3.2mm_M3, F.Cu at (131.7, 105.9)
- added REF**: MountingHole_3.2mm_M3, MountingHole:MountingHole_3.2mm_M3, F.Cu at (139.0, 118.0)
- added SW1: SW_Push, Button_Switch_SMD:SW_DIP_SPSTx01_Slide_6.7x4.1mm_W8.61mm_P2.54mm_LowProfile, F.Cu at (139.0, 107.3)
Routing:
- net Net-(R1-Pad1): track 0.00 -> 9.96 mm
- net Net-(D1-A): track 0.00 -> 1.87 mm
- net GND: track 0.00 -> 1.74 mm, vias 0 -> 1
- added copper zone on F.Cu, net +3V3
- added copper zone on B.Cu, net GND
Other:
- board outline added: 15 x 21 mm
