File: Hardware/kyshi2_horns/kyshi2_horns.kicad_pcb (KiCad board)
At the start: 2 copper layers, 0 parts

Commit message: Horns Board Finished
Parts:
- added C1: 0.1uF, Capacitor_SMD:C_0201_0603Metric_Pad0.64x0.40mm_HandSolder, F.Cu at (119.0, 79.0)
- added C2: 0.1uF, Capacitor_SMD:C_0201_0603Metric_Pad0.64x0.40mm_HandSolder, F.Cu at (129.0, 78.5)
- added C3: 0.1uF, Capacitor_SMD:C_0201_0603Metric_Pad0.64x0.40mm_HandSolder, F.Cu at (133.9, 86.0)
- added C4: 0.1uF, Capacitor_SMD:C_0201_0603Metric_Pad0.64x0.40mm_HandSolder, F.Cu at (126.4, 74.0)
- added C5: 1uF, Capacitor_SMD:C_0201_0603Metric_Pad0.64x0.40mm_HandSolder, F.Cu at (126.5, 76.5)
- added C6: 1uF, Capacitor_SMD:C_0201_0603Metric_Pad0.64x0.40mm_HandSolder, F.Cu at (129.0, 76.0)
- added C7: 10uF, Capacitor_SMD:C_0201_0603Metric_Pad0.64x0.40mm_HandSolder, F.Cu at (135.5, 87.0)
- added C8: 10uF, Capacitor_SMD:C_0201_0603Metric_Pad0.64x0.40mm_HandSolder, F.Cu at (131.5, 87.0)
- added C9: 100uF, Capacitor_SMD:C_0201_0603Metric_Pad0.64x0.40mm_HandSolder, F.Cu at (115.0, 79.0)
- added D1: D, Diode_SMD:D_SMA, F.Cu at (139.5, 74.0)
- added D2: LED, layout:LED_0603_Symbol_on_F.SilkS, F.Cu at (126.8, 87.5)
- added D3: LED, layout:LED_0603_Symbol_on_F.SilkS, F.Cu at (134.5, 78.0)
- added F1: 2A, layout:Fuse_1206_3216Metric, F.Cu at (131.5, 76.0)
- added F2: 2A, layout:Fuse_1206_3216Metric, F.Cu at (114.0, 70.5)
- added J1: Power_Conn, Connector_Molex:Molex_KK-254_AE-6410-03A_1x03_P2.54mm_Vertical, F.Cu at (139.5, 83.5)
- added J2: Horn_In, Connector_Molex:Molex_KK-254_AE-6410-02A_1x02_P2.54mm_Vertical, F.Cu at (117.0, 69.4)
- added J3: Horn_Out_1, Connector_Molex:Molex_KK-254_AE-6410-02A_1x02_P2.54mm_Vertical, F.Cu at (124.1, 69.4)
- added J4: Horn_Out_2, Connector_Molex:Molex_KK-254_AE-6410-02A_1x02_P2.54mm_Vertical, F.Cu at (131.3, 69.4)
- added Q1: Q_NMOS_GDS, Package_TO_SOT_SMD:TO-252-3_TabPin2, F.Cu at (126.6, 82.5)
- added R1: 1k, Resistor_SMD:R_0603_1608Metric_Pad0.98x0.95mm_HandSolder, F.Cu at (119.0, 80.5)
- added R2: 2k, Resistor_SMD:R_0603_1608Metric_Pad0.98x0.95mm_HandSolder, F.Cu at (123.0, 87.5)
- added R3: 2k, Resistor_SMD:R_0603_1608Metric_Pad0.98x0.95mm_HandSolder, F.Cu at (134.5, 82.0)
- added REF**: MountingHole_3.2mm_M3, MountingHole:MountingHole_3.2mm_M3, F.Cu at (117.0, 85.0)
- added REF**: MountingHole_3.2mm_M3, MountingHole:MountingHole_3.2mm_M3, F.Cu at (140.0, 68.5)
- added SW1: SW_Push, Button_Switch_SMD:SW_DIP_SPSTx01_Slide_6.7x4.1mm_W8.61mm_P2.54mm_LowProfile, F.Cu at (119.5, 76.0)
- added TP1: TestPoint, TestPoint:TestPoint_Keystone_5019_Minature, F.Cu at (139.5, 87.0)
Routing:
- net /Horn Control: track 0.00 -> 23.0 mm
- net /Horn In: track 0.00 -> 17.7 mm
- net Net-(Q1-G): track 0.00 -> 16.4 mm, vias 0 -> 2
- net Net-(Q1-D): track 0.00 -> 12.5 mm
- net Net-(J3-Pin_1): track 0.00 -> 10.8 mm
- net Net-(D2-A): track 0.00 -> 4.29 mm
- net Net-(D3-A): track 0.00 -> 2.29 mm
- net Net-(C1-Pad1): track 0.00 -> 2.05 mm
- net GND: vias 0 -> 13
- added copper zone on F.Cu, net +24V
- added copper zone on B.Cu, net GND
Other:
- board outline added: 31.5 x 24.5 mm
