File: Hardware/kyshi2_horns/kyshi2_horns.kicad_sch (KiCad schematic)
At the start: 0 parts

Commit message: Horns Board Finished
Parts:
- added C1, C2, C3, C4: 0.1uF, Capacitor_SMD:C_0201_0603Metric_Pad0.64x0.40mm_HandSolder, symbol device:C
- added C5, C6: 1uF, Capacitor_SMD:C_0201_0603Metric_Pad0.64x0.40mm_HandSolder, symbol device:C
- added C7, C8: 10uF, Capacitor_SMD:C_0201_0603Metric_Pad0.64x0.40mm_HandSolder, symbol device:C
- added C9: 100uF, Capacitor_SMD:C_0201_0603Metric_Pad0.64x0.40mm_HandSolder, symbol device:C
- added D1: D, Diode_SMD:D_SMA, symbol Device:D
- added D2, D3: LED, layout:LED_0603_Symbol_on_F.SilkS, symbol device:LED
- added F1, F2: 2A, layout:Fuse_1206_3216Metric, symbol device:Fuse
- added J1: Power_Conn, Connector_Molex:Molex_KK-254_AE-6410-03A_1x03_P2.54mm_Vertical, symbol Connector_Generic:Conn_01x03
- added J2: Horn_In, Connector_Molex:Molex_KK-254_AE-6410-02A_1x02_P2.54mm_Vertical, symbol Connector_Generic:Conn_01x02
- added J3: Horn_Out_1, Connector_Molex:Molex_KK-254_AE-6410-02A_1x02_P2.54mm_Vertical, symbol Connector_Generic:Conn_01x02
- added J4: Horn_Out_2, Connector_Molex:Molex_KK-254_AE-6410-02A_1x02_P2.54mm_Vertical, symbol Connector_Generic:Conn_01x02
- added Q1: Q_NMOS_GDS, Package_TO_SOT_SMD:TO-252-3_TabPin2, symbol device:Q_NMOS_GDS
- added R1: 1k, Resistor_SMD:R_0603_1608Metric_Pad0.98x0.95mm_HandSolder, symbol Device:R_US
- added R2, R3: 2k, Resistor_SMD:R_0603_1608Metric_Pad0.98x0.95mm_HandSolder, symbol Device:R_US
- added SW1: SW_Push, Button_Switch_SMD:SW_DIP_SPSTx01_Slide_6.7x4.1mm_W8.61mm_P2.54mm_LowProfile, symbol Switch:SW_Push
- added TP1: TestPoint, TestPoint:TestPoint_Keystone_5019_Minature, symbol Connector:TestPoint
Connections:
- new net: J3.1 (Pin_1), J4.2 (Pin_2)
- new net: D2.2 (A), R2.1
- new net: F2.1, Q1.1 (G), R1.1
- new net: F1.2, Q1.2 (D)
- new net: D3.2 (A), R3.1
- new net: C1.1, R1.2
- new net +24V: C2.2, C3.2, C4.2, C5.2, C6.2, C7.2, C8.2, C9.2, D1.1 (K), J1.2 (Pin_2), J3.2 (Pin_2), R3.2, SW1.2, TP1.1
- new net GND: C1.2, C2.1, C3.1, C4.1, C5.1, C6.1, C7.1, C8.1, C9.1, D2.1 (K), J1.1 (Pin_1), J1.3 (Pin_3), J2.2 (Pin_2), Q1.3 (S)
- new net Horn Control: F2.2, J2.1 (Pin_1), R2.2, SW1.1
- new net Horn In: D1.2 (A), D3.1 (K), F1.1, J4.1 (Pin_1)
Other:
- title: Template -> Horns Board
