File: Hardware/jerrywang_Horns_v1.0/jerrywang_Horns_v1.0.kicad_pcb (KiCad board)
At the start: 2 copper layers, 0 parts

Commit message: Solar Car Onboarding Complete
Parts:
- added C1: 0.1µF, Capacitor_SMD:C_1206_3216Metric, F.Cu at (111.1, 78.0)
- added C2: 0.1µF, Capacitor_SMD:C_1206_3216Metric, F.Cu at (111.3, 83.4)
- added C3: 0.1µF, Capacitor_SMD:C_1206_3216Metric, F.Cu at (111.4, 88.7)
- added C4: 0.1µF, Capacitor_SMD:C_1206_3216Metric, F.Cu at (111.5, 94.6)
- added C5: 1µF, Capacitor_SMD:C_1206_3216Metric, F.Cu at (111.1, 100.5)
- added C6: 1µF, Capacitor_SMD:C_1206_3216Metric, F.Cu at (111.1, 105.8)
- added C7: 10µF, Capacitor_SMD:C_1206_3216Metric, F.Cu at (111.1, 111.4)
- added C8: 10µF, Capacitor_SMD:C_1206_3216Metric, F.Cu at (110.8, 118.1)
- added C9: 100µF_Polarized, Capacitor_THT:CP_Radial_D8.0mm_P3.50mm, F.Cu at (119.4, 111.5)
- added D1: ES2DA-13-F, Diode_SMD:D_SMA, F.Cu at (135.8, 91.3)
- added F1: 2A, Fuse:Fuse_1206_3216Metric, F.Cu at (136.1, 98.9)
- added Horn#1: Conn_01x02, Connector_PinSocket_2.54mm:PinSocket_1x02_P2.54mm_Vertical, F.Cu at (118.6, 79.4)
- added Horn#2: Conn_01x02, Connector_PinSocket_2.54mm:PinSocket_1x02_P2.54mm_Vertical, F.Cu at (127.3, 83.1)
- added HornControl1: Conn_01x02, Connector_PinSocket_2.54mm:PinSocket_1x02_P2.54mm_Vertical, F.Cu at (137.6, 79.3)
- added J1: Conn_01x03, Connector_PinSocket_2.54mm:PinSocket_1x03_P2.54mm_Vertical, F.Cu at (131.8, 105.4)
- added Q2: IRFR010PBF, Package_TO_SOT_SMD:TO-252-2, F.Cu at (123.5, 97.1)
- added R1: 1K, Resistor_SMD:R_1206_3216Metric, F.Cu at (138.3, 108.0)
Routing:
- net GND: track 0.00 -> 87.1 mm, vias 0 -> 4
- net /HORN_CTL: track 0.00 -> 82.0 mm
- net +24V: track 0.00 -> 58.3 mm, vias 0 -> 2
- net /HORN_IN: track 0.00 -> 24.1 mm
- net Net-(Horn#2-Pin_2): track 0.00 -> 16.3 mm
- net Net-(Horn#1-Pin_2): track 0.00 -> 9.18 mm
- added copper zone on F.Cu, net +24V
- added copper zone on B.Cu, net GND
Other:
- board outline added: 43 x 55.7 mm
