File: hw-horns/hw-horns.kicad_pcb (KiCad board)
At the start: 2 copper layers, 17 parts, among them J1 Conn_01x03_Female, J2 Conn_01x02_Female, J3 Conn_01x02_Male, J4 Conn_01x02_Male, Q1 IRFS4127

Commit message: Finished PCB for horns project
Parts:
- added REF**: MountingHole_2.1mm, MountingHole:MountingHole_2.1mm, F.Cu at (150.5, 113.8)
- added REF**: MountingHole_2.1mm, MountingHole:MountingHole_2.1mm, F.Cu at (149.0, 94.5)
- added REF**: MountingHole_2.1mm, MountingHole:MountingHole_2.1mm, F.Cu at (185.2, 113.8)
- added REF**: MountingHole_2.1mm, MountingHole:MountingHole_2.1mm, F.Cu at (186.5, 95.0)
- moved J3 2.54 mm to (176.5, 97.5), turned to -90 degrees
- moved J4 2.52 mm to (176.5, 107.5), turned to -90 degrees
- moved C1 1.88 mm to (152.5, 89.0), turned to -90 degrees
- moved Q1 0.47 mm to (165.0, 102.9)
- moved C2 0.12 mm to (158.2, 90.1), turned to -90 degrees
- moved C3 0.12 mm to (162.5, 90.1), turned to -90 degrees
- moved C7 0.12 mm to (180.8, 89.8), turned to -90 degrees
- moved C8 0.12 mm to (185.8, 89.8), turned to -90 degrees
- moved C4 0.06 mm to (167.5, 89.9), turned to -90 degrees
- turned C5 to -90 degrees
- turned C6 to -90 degrees
- turned D1 to -90 degrees
- turned F1 to 180 degrees
- turned R1 to -90 degrees
Routing:
- net GND: track 0.00 -> 63.2 mm, vias 0 -> 2
- net +24V: track 0.00 -> 43.8 mm
- net /Horn Control: track 0.00 -> 28.0 mm
- net Net-(Q1-D): track 0.00 -> 20.3 mm
- net /Horn In: track 0.00 -> 19.2 mm
- net Net-(J3-Pin_2): track 0.00 -> 7.47 mm
- added copper zone on F.Cu, net +24V
- added copper zone on B.Cu, net GND
Other:
- board outline added: 45.2 x 32.9 mm

Commit message: fixed use of vias in PCB horns
Parts:
- moved C1 0.50 mm to (152.5, 88.5)
Routing:
- net GND: track 63.2 -> 51.3 mm
- net /Horn Control: track 28.0 -> 37.2 mm
Changed lines of the file:
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@@
 	(footprint "Capacitor_THT:CP_Radial_D4.0mm_P2.00mm"
 		(layer "F.Cu")
-		(at 152.5 89.027401 -90)
+		(at 152.5 88.527401 -90)
 		(descr "CP, Radial series, Radial, pin pitch=2.00mm, , diameter=4mm, Electrolytic Capacitor")
 		(tags "CP Radial series Radial pin pitch 2.00mm  diameter 4mm Electrolytic Capacitor")
@@
 	)
 	(segment
+		(start 158.222599 88.527401)
+		(end 158.25 88.5)
+		(width 0.25)
+		(layer "F.Cu")
+		(net 1)
+	)
+	(segment
 		(start 162.5 88.5)
 		(end 167.375 88.5)
@@
 	)
 	(segment
+		(start 152.5 88.527401)
+		(end 158.222599 88.527401)
+		(width 0.25)
+		(layer "F.Cu")
+		(net 1)
+	)
+	(segment
 		(start 176.375 88.375)
 		(end 176.5 88.25)
@@
 	)
 	(segment
-		(start 154.722599 89.027401)
-		(end 155.25 88.5)
-		(width 0.25)
-		(layer "F.Cu")
-		(net 1)
-	)
-	(segment
-		(start 155.25 88.5)
-		(end 158.25 88.5)
-		(width 0.25)
-		(layer "F.Cu")
-		(net 1)
-	)
-	(segment
 		(start 176.5 88.25)
 		(end 180.75 88.25)
@@
 	)
 	(segment
-		(start 152.5 89.027401)
-		(end 154.722599 89.027401)
+		(start 167.28 109.22)
+		(end 167.25 109.25)
 		(width 0.25)
 		(layer "F.Cu")
-		(net 1)
+		(net 2)
 	)
 	(segment
-		(start 154.5 94)
-		(end 154.5 93.027401)
+		(start 158.25 91.625)
+		(end 153.597598 91.625)
 		(width 0.25)
 		(layer "F.Cu")
@@
 	)
 	(segment
-		(start 160.5 110.5)
-		(end 160.5 110.54)
+		(start 167.28 107.125)
+		(end 167.28 109.22)
 		(width 0.25)
 		(layer "F.Cu")
@@
 	)
 	(segment
-		(start 152.5 91.027401)
-		(end 157.652401 91.027401)
-		(width 0.25)
-		(layer "F.Cu")
-		(net 2)
-	)
-	(segment
-		(start 160.5 110)
-		(end 160.5 110.5)
-		(width 0.25)
-		(layer "F.Cu")
-		(net 2)
-	)
-	(segment
-		(start 156.5 112.75)
-		(end 157.25 112.75)
-		(width 0.25)
-		(layer "F.Cu")
-		(net 2)
-	)
-	(segment
-		(start 160.5 110.54)
-		(end 163.71 113.75)
+		(start 153.597598 91.625)
+		(end 152.5 90.527401)
 		(width 0.25)
 		(layer "F.Cu")
@@
 	)
 	(segment
-		(start 163.71 113.75)
-		(end 163.71 110.695)
-		(width 0.25)
-		(layer "F.Cu")
-		(net 2)
-	)
-	(segment
-		(start 163.71 110.695)
-		(end 167.28 107.125)
+		(start 156.5 110.25)
+		(end 158.5 110.25)
 		(width 0.25)
 		(layer "F.Cu")
@@
 	)
 	(segment
-		(start 157.25 112.75)
-		(end 158.25 113.75)
-		(width 0.25)
-		(layer "F.Cu")
-		(net 2)
-	)
-	(segment
-		(start 154.5 93.027401)
-		(end 152.5 91.027401)
-		(width 0.25)
-		(layer "F.Cu")
-		(net 2)
-	)
-	(segment
 		(start 180.625 91.5)
 		(end 180.75 91.375)
@@
 	)
 	(segment
+		(start 158.5 110.25)
+		(end 158.5 112.75)
+		(width 0.25)
+		(layer "F.Cu")
+		(net 2)
+	)
+	(segment
 		(start 163.25 91.75)
 		(end 163.4375 91.5625)
@@
 	)
 	(segment
+		(start 156.5 112.75)
+		(end 158.5 112.75)
+		(width 0.25)
+		(layer "F.Cu")
+		(net 2)
+	)
+	(segment
 		(start 180.75 91.375)
 		(end 185.75 91.375)
@@
 	)
 	(segment
-		(start 167.5 91.5)
-		(end 171.75 91.5)
+		(start 158.5 112.75)
+		(end 158.5 115.75)
 		(width 0.25)
 		(layer "F.Cu")
@@
 	)
 	(segment
-		(start 158.25 91.625)
-		(end 162.5 91.625)
+		(start 167.5 91.5)
+		(end 171.75 91.5)
 		(width 0.25)
 		(layer "F.Cu")
@@
 	)
 	(segment
-		(start 158.25 113.75)
-		(end 163.71 113.75)
+		(start 158.25 91.625)
+		(end 162.5 91.625)
 		(width 0.25)
 		(layer "F.Cu")
@@
 	)
 	(via
-		(at 160.5 110)
+		(at 167.25 109.25)
 		(size 0.8)
 		(drill 0.4)
@@
 	)
 	(via
-		(at 154.5 94)
+		(at 158.5 115.75)
 		(size 0.8)
 		(drill 0.4)
@@
 	)
 	(segment
+		(start 166.25 111)
+		(end 165 109.75)
+		(width 0.25)
+		(layer "F.Cu")
+		(net 3)
+	)
+	(segment
+		(start 161.5 115.75)
+		(end 160.5 116.75)
+		(width 0.25)
+		(layer "F.Cu")
+		(net 3)
+	)
+	(segment
 		(start 156.5 108.425)
 		(end 155.575 108.425)
@@
 	)
 	(segment
+		(start 165 109.75)
+		(end 161.5 109.75)
+		(width 0.25)
+		(layer "F.Cu")
+		(net 3)
+	)
+	(segment
 		(start 156.5 108.425)
 		(end 156.575 108.425)
@@
 	)
 	(segment
-		(start 164.125 115.875)
-		(end 166.25 113.75)
+		(start 160.5 116.75)
+		(end 157.375 116.75)
 		(width 0.25)
 		(layer "F.Cu")
@@
 	)
 	(segment
-		(start 156.5 115.875)
-		(end 164.125 115.875)
+		(start 166.25 113.75)
+		(end 166.25 111)
+		(width 0.25)
+		(layer "F.Cu")
+		(net 3)
+	)
+	(segment
+		(start 161.5 109.75)
+		(end 161.5 115.75)
+		(width 0.25)
+		(layer "F.Cu")
+		(net 3)
+	)
+	(segment
+		(start 157.375 116.75)
+		(end 156.5 115.875)
 		(width 0.25)
 		(layer "F.Cu")
@@
 		(end 176.5 107.48)
 		(width 0.25)
-		(layer "B.Cu")
+		(layer "F.Cu")
+		(net 6)
+	)
+	(segment
+		(start 176.5 107.48)
+		(end 176.52 107.5)
+		(width 0.25)
+		(layer "F.Cu")
 		(net 6)
 	)
