File: hw-horns/hw-horns.kicad_sch (KiCad schematic)
At the start: 17 parts, among them J1 Conn_01x03_Female, J2 Conn_01x02_Female, J3 Conn_01x02_Male, J4 Conn_01x02_Male, Q1 IRFS4127

Commit message: Finished PCB for horns project
Other:
- moved on the sheet: J2
Changed lines of the file:
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@@
 	(wire
 		(pts
-			(xy 149.86 132.08) (xy 149.86 148.59)
+			(xy 149.86 132.08) (xy 149.86 137.16)
 		)
 		(stroke
@@
 	(wire
 		(pts
-			(xy 152.4 128.27) (xy 152.4 148.59)
+			(xy 152.4 128.27) (xy 152.4 137.16)
 		)
 		(stroke
@@
 	(symbol
 		(lib_id "Connector:Conn_01x02_Female")
-		(at 152.4 153.67 270)
+		(at 152.4 142.24 270)
 		(unit 1)
 		(exclude_from_sim no)
@@
 		(fields_autoplaced yes)
 		(property "Reference" "J2"
-			(at 148.59 154.3051 90)
+			(at 148.59 142.8751 90)
 			(effects
 				(font
@@
 		)
 		(property "Value" "Conn_01x02_Female"
-			(at 148.59 151.7651 90)
+			(at 148.59 140.3351 90)
 			(effects
 				(font
@@
 		)
 		(property "Footprint" "Connector_Molex:Molex_KK-254_AE-6410-02A_1x02_P2.54mm_Vertical"
-			(at 152.4 153.67 0)
+			(at 152.4 142.24 0)
 			(effects
 				(font
@@
 		)
 		(property "Datasheet" "~"
-			(at 152.4 153.67 0)
+			(at 152.4 142.24 0)
 			(effects
 				(font
@@
 		)
 		(property "Description" "Generic connector, single row, 01x02, script generated (kicad-library-utils/schlib/autogen/connector/)"
-			(at 152.4 153.67 0)
-			(effects
-				(font
+			(at 152.4 142.24 0)
+			(effects
+				(font

Commit message: Fixed connectors on schematic to generic
Parts:
- removed J1: Conn_01x03_Female, Connector_Molex:Molex_KK-254_AE-6410-03A_1x03_P2.54mm_Vertical, symbol Connector:Conn_01x03_Female
- removed J2: Conn_01x02_Female, Connector_Molex:Molex_KK-254_AE-6410-02A_1x02_P2.54mm_Vertical, symbol Connector:Conn_01x02_Female
- removed J3, J4: Conn_01x02_Male, Connector_Molex:Molex_KK-254_AE-6410-02A_1x02_P2.54mm_Vertical, symbol Connector:Conn_01x02_Male
- added J1, J2, J3: Conn_01x02, Connector_Molex:Molex_KK-254_AE-6410-02A_1x02_P2.54mm_Vertical, symbol Connector_Generic:Conn_01x02
- added J5: Conn_01x03, Connector_Molex:Molex_KK-254_AE-6410-03A_1x03_P2.54mm_Vertical, symbol Connector_Generic:Conn_01x03
Connections:
- net +24V: now also J2.1 (Pin_1), J5.2 (Pin_2)
- net GND: now also J1.1 (Pin_1), J5.1 (Pin_1), J5.3 (Pin_3)
- net Horn Control: now also J1.2 (Pin_2)
- net Horn In: now also J3.2 (Pin_2)
- new net: J2.2 (Pin_2), J3.1 (Pin_1)
