File: Hardware/tkiran2_horns/horn_v0.0.kicad_pcb (KiCad board)
At the start: 2 copper layers, 0 parts

Commit message: tkiran2_onboarding
Parts:
- added C1: 1uF, Capacitor_SMD:C_0603_1608Metric_Pad1.08x0.95mm_HandSolder, F.Cu at (147.9, 108.0)
- added C2: .1uF, Capacitor_SMD:C_0603_1608Metric_Pad1.08x0.95mm_HandSolder, F.Cu at (126.0, 93.0)
- added C3: .1uF, Capacitor_SMD:C_0603_1608Metric_Pad1.08x0.95mm_HandSolder, F.Cu at (126.0, 95.5)
- added C4: .1uF, Capacitor_SMD:C_0603_1608Metric_Pad1.08x0.95mm_HandSolder, F.Cu at (126.0, 98.0)
- added C5: 1uF, Capacitor_SMD:C_0603_1608Metric_Pad1.08x0.95mm_HandSolder, F.Cu at (126.0, 100.5)
- added C6: 1uF, Capacitor_SMD:C_0603_1608Metric_Pad1.08x0.95mm_HandSolder, F.Cu at (126.0, 103.0)
- added C7: 10uF, Capacitor_SMD:C_0603_1608Metric_Pad1.08x0.95mm_HandSolder, F.Cu at (126.0, 105.5)
- added C8: 10uF, Capacitor_SMD:C_0603_1608Metric_Pad1.08x0.95mm_HandSolder, F.Cu at (126.0, 108.0)
- added C9: 100uF, Capacitor_SMD:C_Elec_5x5.8, F.Cu at (141.9, 106.5)
- added D1: S2JTR, Diode_SMD:D_SMB, F.Cu at (132.3, 109.5)
- added F1: 2A, Fuse:Fuse_0603_1608Metric_Pad1.05x0.95mm_HandSolder, F.Cu at (146.0, 112.0)
- added J1: Conn_01x03, Connector_JST:JST_EH_B3B-EH-A_1x03_P2.50mm_Vertical, F.Cu at (141.2, 99.9)
- added J2: Conn_01x02, Connector_JST:JST_EH_B2B-EH-A_1x02_P2.50mm_Vertical, F.Cu at (131.7, 91.8)
- added J3: Conn_01x02, Connector_JST:JST_EH_B2B-EH-A_1x02_P2.50mm_Vertical, F.Cu at (131.7, 97.7)
- added J4: Conn_01x02, Connector_JST:JST_EH_B2B-EH-A_1x02_P2.50mm_Vertical, F.Cu at (131.7, 103.5)
- added Q1: STD7NK40Z, Package_TO_SOT_SMD:TO-252-2, F.Cu at (143.8, 93.2)
- added R1: 1k, Resistor_SMD:R_0201_0603Metric_Pad0.64x0.40mm_HandSolder, F.Cu at (147.6, 104.0)
- added REF**: MountingHole_3.2mm_M3, MountingHole:MountingHole_3.2mm_M3, F.Cu at (120.0, 110.0)
- added REF**: MountingHole_3.2mm_M3, MountingHole:MountingHole_3.2mm_M3, F.Cu at (120.0, 93.0)
- added REF**: MountingHole_3.2mm_M3, MountingHole:MountingHole_3.2mm_M3, F.Cu at (153.0, 110.0)
- added REF**: MountingHole_3.2mm_M3, MountingHole:MountingHole_3.2mm_M3, F.Cu at (153.0, 93.0)
Routing:
- net Net-(Q1-D): track 0.00 -> 24.6 mm
- net +24V: track 0.00 -> 22.5 mm, vias 0 -> 7
- net /HORN_IN: track 0.00 -> 22.4 mm
- net GND: track 0.00 -> 13.6 mm, vias 0 -> 9
- net Net-(D1-K): track 0.00 -> 12.5 mm
- net Net-(J3-Pin_2): track 0.00 -> 6.89 mm
- added copper zone on B.Cu, net +24V
- added copper zone on F.Cu, net +24V
- added copper zone on B.Cu, net GND
Other:
- board outline added: 43 x 25 mm

Commit message: horns
Parts:
- turned F1 to 180 degrees
Routing:
- net +24V: track 22.5 -> 13.5 mm, vias 7 -> 0
- net /HORN_IN: track 22.4 -> 20.4 mm
- net Net-(Q1-D): track 24.6 -> 22.7 mm
- removed copper zone on B.Cu, net +24V
Changed lines of the file:
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@@
 	(footprint "Fuse:Fuse_0603_1608Metric_Pad1.05x0.95mm_HandSolder"
 		(layer "F.Cu")
-		(at 146 112)
+		(at 146 112 180)
 		(descr "Fuse SMD 0603 (1608 Metric), square (rectangular) end terminal, IPC_7351 nominal with elongated pad for handsoldering. (Body size source: http://www.tortai-tech.com/upload/download/2011102023233369053.pdf), generated with kicad-footprint-generator")
 		(tags "fuse handsolder")
@@
 		(attr smd)
 		(fp_line
+			(start -0.171267 0.51)
+			(end 0.171267 0.51)
+			(stroke
+				(width 0.12)
+				(type solid)
+			)
+			(layer "F.SilkS")
+		)
+		(fp_line
 			(start -0.171267 -0.51)
 			(end 0.171267 -0.51)
@@
 		)
 		(fp_line
-			(start -0.171267 0.51)
-			(end 0.171267 0.51)
-			(stroke
-				(width 0.12)
-				(type solid)
-			)
-			(layer "F.SilkS")
+			(start 1.65 0.73)
+			(end -1.65 0.73)
+			(stroke
+				(width 0.05)
+				(type solid)
+			)
+			(layer "F.CrtYd")
+		)
+		(fp_line
+			(start 1.65 -0.73)
+			(end 1.65 0.73)
+			(stroke
+				(width 0.05)
+				(type solid)
+			)
+			(layer "F.CrtYd")
+		)
+		(fp_line
+			(start -1.65 0.73)
+			(end -1.65 -0.73)
+			(stroke
+				(width 0.05)
+				(type solid)
+			)
+			(layer "F.CrtYd")
 		)
 		(fp_line
@@
 		)
 		(fp_line
-			(start -1.65 0.73)
-			(end -1.65 -0.73)
-			(stroke
-				(width 0.05)
-				(type solid)
-			)
-			(layer "F.CrtYd")
-		)
-		(fp_line
-			(start 1.65 -0.73)
-			(end 1.65 0.73)
-			(stroke
-				(width 0.05)
-				(type solid)
-			)
-			(layer "F.CrtYd")
-		)
-		(fp_line
-			(start 1.65 0.73)
-			(end -1.65 0.73)
-			(stroke
-				(width 0.05)
-				(type solid)
-			)
-			(layer "F.CrtYd")
+			(start 0.8 0.4)
+			(end -0.8 0.4)
+			(stroke
+				(width 0.1)
+				(type solid)
+			)
+			(layer "F.Fab")
+		)
+		(fp_line
+			(start 0.8 -0.4)
+			(end 0.8 0.4)
+			(stroke
+				(width 0.1)
+				(type solid)
+			)
+			(layer "F.Fab")
+		)
+		(fp_line
+			(start -0.8 0.4)
+			(end -0.8 -0.4)
+			(stroke
+				(width 0.1)
+				(type solid)
+			)
+			(layer "F.Fab")
 		)
 		(fp_line
@@
 			(layer "F.Fab")
 		)
-		(fp_line
-			(start -0.8 0.4)
-			(end -0.8 -0.4)
-			(stroke
-				(width 0.1)
-				(type solid)
-			)
-			(layer "F.Fab")
-		)
-		(fp_line
-			(start 0.8 -0.4)
-			(end 0.8 0.4)
-			(stroke
-				(width 0.1)
-				(type solid)
-			)
-			(layer "F.Fab")
-		)
-		(fp_line
-			(start 0.8 0.4)
-			(end -0.8 0.4)
-			(stroke
-				(width 0.1)
-				(type solid)
-			)
-			(layer "F.Fab")
-		)
 		(fp_text user "${REFERENCE}"
 			(at 0 0 0)
@@
 		)
 		(pad "1" smd roundrect
-			(at -0.875 0)
+			(at -0.875 0 180)
 			(size 1.05 0.95)
 			(layers "F.Cu" "F.Mask" "F.Paste")
@@
 		)
 		(pad "2" smd roundrect
-			(at 0.875 0)
+			(at 0.875 0 180)
 			(size 1.05 0.95)
 			(layers "F.Cu" "F.Mask" "F.Paste")
@@
 	)
 	(segment
-		(start 123.86 105.54)
-		(end 123.825 105.575)
-		(width 0.25)
-		(layer "F.Cu")
-		(net 4)
-	)
-	(segment
-		(start 123.89 98.01)
-		(end 123.85 98.05)
-		(width 0.25)
-		(layer "F.Cu")
-		(net 4)
-	)
-	(segment
-		(start 125.125 100.52)
-		(end 123.83 100.52)
-		(width 0.25)
-		(layer "F.Cu")
-		(net 4)
-	)
-	(segment
-		(start 125.125 95.5)
-		(end 123.925 95.5)
-		(width 0.25)
-		(layer "F.Cu")
-		(net 4)
-	)
-	(segment
 		(start 143.7375 99.9)
 		(end 134.4875 109.15)
@@
 	)
 	(segment
-		(start 123.925 95.5)
-		(end 123.875 95.45)
-		(width 0.25)
-		(layer "F.Cu")
-		(net 4)
-	)
-	(segment
-		(start 125.125 108.05)
-		(end 123.875 108.05)
-		(width 0.25)
-		(layer "F.Cu")
-		(net 4)
-	)
-	(segment
-		(start 124.085 92.99)
-		(end 123.95 93.125)
-		(width 0.25)
-		(layer "F.Cu")
-		(net 4)
-	)
-	(segment
-		(start 123.895 103.03)
-		(end 123.85 103.075)
-		(width 0.25)
-		(layer "F.Cu")
-		(net 4)
-	)
-	(segment
-		(start 125.125 98.01)
-		(end 123.89 98.01)
-		(width 0.25)
-		(layer "F.Cu")
-		(net 4)
-	)
-	(segment
-		(start 125.125 92.99)
-		(end 124.085 92.99)
-		(width 0.25)
-		(layer "F.Cu")
-		(net 4)
-	)
-	(segment
-		(start 123.83 100.52)
-		(end 123.825 100.525)
-		(width 0.25)
-		(layer "F.Cu")
-		(net 4)
-	)
-	(segment
-		(start 125.125 103.03)
-		(end 123.895 103.03)
-		(width 0.25)
-		(layer "F.Cu")
-		(net 4)
-	)
-	(segment
-		(start 123.875 108.05)
-		(end 123.825 108.1)
-		(width 0.25)
-		(layer "F.Cu")
-		(net 4)
-	)
-	(segment
-		(start 125.125 105.54)
-		(end 123.86 105.54)
-		(width 0.25)
-		(layer "F.Cu")
-		(net 4)
-	)
-	(via
-		(at 123.825 108.1)
-		(size 0.8)
-		(drill 0.4)
-		(layers "F.Cu" "B.Cu")
-		(free yes)
-		(net 4)
-	)
-	(via
-		(at 123.85 98.05)
-		(size 0.8)
-		(drill 0.4)
-		(layers "F.Cu" "B.Cu")
-		(free yes)
-		(net 4)
-	)
-	(via
-		(at 123.825 100.525)
-		(size 0.8)
-		(drill 0.4)
-		(layers "F.Cu" "B.Cu")
-		(free yes)
-		(net 4)
-	)
-	(via
-		(at 123.95 93.125)
-		(size 0.8)
-		(drill 0.4)
-		(layers "F.Cu" "B.Cu")
-		(free yes)
-		(net 4)
-	)
-	(via
-		(at 123.85 103.075)
-		(size 0.8)
-		(drill 0.4)
-		(layers "F.Cu" "B.Cu")
-		(free yes)
-		(net 4)
-	)
-	(via
-		(at 123.875 95.45)
-		(size 0.8)
-		(drill 0.4)
-		(layers "F.Cu" "B.Cu")
-		(free yes)
-		(net 4)
-	)
-	(via
-		(at 123.825 105.575)
-		(size 0.8)
-		(drill 0.4)
-		(layers "F.Cu" "B.Cu")
-		(free yes)
-		(net 4)
-	)
-	(segment
 		(start 130.1875 99.2)
 		(end 130.1875 109.55)
@@
 	)
 	(segment
-		(start 132.9125 111.025)
-		(end 145.9 111.025)
+		(start 134.205698 112.318198)
+		(end 144.806802 112.318198)
+		(width 0.25)
+		(layer "F.Cu")
+		(net 6)
+	)
+	(segment
+		(start 132.9125 104.825)
+		(end 132.9125 111.025)
 		(width 0.25)
 		(layer "F.Cu")
@@
 	)
 	(segment
-		(start 132.9125 104.825)
-		(end 132.9125 111.025)
+		(start 132.9125 111.025)
+		(end 134.205698 112.318198)
 		(width 0.25)
 		(layer "F.Cu")
@@
 	)
 	(segment
-		(start 145.9 111.025)
+		(start 151.125 98.4875)
+		(end 151.125 107.75)
+		(width 0.25)
+		(layer "F.Cu")
+		(net 7)
+	)
+	(segment
+		(start 151.125 107.75)
 		(end 146.875 112)
 		(width 0.25)
 		(layer "F.Cu")
-		(net 6)
-	)
-	(segment
-		(start 145.925 112.8)
-		(end 145.125 112)
-		(width 0.25)
-		(layer "F.Cu")
 		(net 7)
 	)
 	(segment
-		(start 147.402076 112.8)
-		(end 145.925 112.8)
-		(width 0.25)
-		(layer "F.Cu")
-		(net 7)
-	)
-	(segment
 		(start 145.8875 93.25)
-		(end 149.5875 96.95)
-		(width 0.25)
-		(layer "F.Cu")
-		(net 7)
-	)
-	(segment
-		(start 149.5875 96.95)
-		(end 149.5875 110.614576)
-		(width 0.25)
-		(layer "F.Cu")
-		(net 7)
-	)
-	(segment
-		(start 149.5875 110.614576)
-		(end 147.402076 112.8)
+		(end 151.125 98.4875)
 		(width 0.25)
 		(layer "F.Cu")
@@
 		(connect_pads
 			(clearance 0.508)
-		)
-		(min_thickness 0.25)
-		(filled_areas_thickness no)
-		(fill yes
-			(thermal_gap 0.5)
-			(thermal_bridge_width 0.5)
-		)
-		(polygon
-			(pts
-				(xy 115 89) (xy 158 89) (xy 158 114) (xy 115 114)
-			)
-		)
-	)
-	(zone
-		(net 4)
-		(net_name "+24V")
-		(layer "B.Cu")
-		(hatch edge 0.5)
-		(priority 2)
-		(connect_pads
-			(clearance 0.508)

Commit message: horns
Routing:
- net /HORN_CTL: track 0.00 -> 25.5 mm
- net Net-(Q1-G): track 0.00 -> 18.2 mm
- net Net-(C1-Pad2): track 0.00 -> 4.31 mm
Changed lines of the file:
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@@
+	)
+	(segment
+		(start 145 99.375799)
+		(end 145 102.761312)
+		(width 0.25)
+		(layer "F.Cu")
+		(net 1)
+	)
+	(segment
+		(start 145 102.761312)
+		(end 147.8625 105.623812)
+		(width 0.25)
+		(layer "F.Cu")
+		(net 1)
+	)
+	(segment
+		(start 134.1875 91.85)
+		(end 134.1875 94.1875)
+		(width 0.25)
+		(layer "F.Cu")
+		(net 1)
+	)
+	(segment
+		(start 138.6 98.6)
+		(end 144.224201 98.6)
+		(width 0.25)
+		(layer "F.Cu")
+		(net 1)
+	)
+	(segment
+		(start 134.1875 94.1875)
+		(end 138.6 98.6)
+		(width 0.25)
+		(layer "F.Cu")
+		(net 1)
+	)
+	(segment
+		(start 147.8625 107.1375)
+		(end 147 108)
+		(width 0.25)
+		(layer "F.Cu")
+		(net 1)
+	)
+	(segment
+		(start 144.224201 98.6)
+		(end 145 99.375799)
+		(width 0.25)
+		(layer "F.Cu")
+		(net 1)
+	)
+	(segment
+		(start 147.8625 105.623812)
+		(end 147.8625 107.1375)
+		(width 0.25)
+		(layer "F.Cu")
+		(net 1)
+	)
+	(segment
+		(start 148.725 104.75)
+		(end 148.725 108)
+		(width 0.25)
+		(layer "F.Cu")
+		(net 2)
+	)
+	(segment
+		(start 147.975 104)
+		(end 148.725 104.75)
+		(width 0.25)
+		(layer "F.Cu")
+		(net 2)
 	)
 	(segment
@@
 		(net 8)
 	)
+	(segment
+		(start 142.3625 93.745)
+		(end 142.3625 97.3625)
+		(width 0.25)
+		(layer "F.Cu")
+		(net 9)
+	)
+	(segment
+		(start 147.16 103.800001)
+		(end 147.16 104)
+		(width 0.25)
+		(layer "F.Cu")
+		(net 9)
+	)
+	(segment
+		(start 139.5875 90.97)
+		(end 142.3625 93.745)
+		(width 0.25)
+		(layer "F.Cu")
+		(net 9)
+	)
+	(segment
+		(start 142.3625 97.3625)
+		(end 145.486701 97.3625)
+		(width 0.25)
+		(layer "F.Cu")
+		(net 9)
+	)
+	(segment
+		(start 147.4125 103.547501)
+		(end 147.16 103.800001)
+		(width 0.25)
+		(layer "F.Cu")
+		(net 9)
+	)
+	(segment
+		(start 147.4125 99.288299)
+		(end 147.4125 103.547501)
+		(width 0.25)
+		(layer "F.Cu")
+		(net 9)
+	)
+	(segment
+		(start 145.486701 97.3625)
+		(end 147.4125 99.288299)
+		(width 0.25)
+		(layer "F.Cu")
+		(net 9)
+	)
 	(zone
