File: Hardware/idwiv_Horns_v1.0(kicad_prl)/idwiv_Horns_v1.0(schematic).kicad_sch (KiCad schematic)
At the start: 6 parts, among them J1 Conn_01x03_MountingPin, J2 Conn_01x03_MountingPin, J3 Conn_01x03_MountingPin, J4 Conn_01x02_Pin, J5 Conn_01x02_Pin, J6 Conn_01x02_Pin

Commit message: completed difficult hardware project
Parts:
- removed J1, J2, J3: Conn_01x03_MountingPin, symbol Connector_Generic_MountingPin:Conn_01x03_MountingPin
- removed J4, J5, J6: Conn_01x02_Pin, symbol Connector:Conn_01x02_Pin
- added C1, C2, C3, C9: 0.1u, symbol Device:C
- added C4, C5: 1u, symbol Device:C
- added C6, C7: 10u, symbol Device:C
- added C8: 100u, symbol Device:C
- added F1: Fuse, symbol Device:Fuse
- added J1: Conn_01x03, symbol Connector_Generic:Conn_01x03
- added J2, J3, J4: Conn_01x02, symbol Connector_Generic:Conn_01x02
- added Q1: IRFS4115, Package_TO_SOT_SMD:TO-263-2, symbol Transistor_FET:IRFS4115
- added R1: R_US, symbol Device:R_US
Connections:
- net +24V: now also J1.2 (Pin_2)
- net GND: now also C1.2, J1.1 (Pin_1), J1.3 (Pin_3), J2.1 (Pin_1), R1.2
- net Horn Control: now also C1.1, J2.2 (Pin_2), Q1.1 (G), R1.1
- net Horn In: now also F1.1, J3.2 (Pin_2)
- new net: F1.2, Q1.2 (D)
- new net: J4.2 (Pin_2), Q1.3 (S)
- new net: J3.1 (Pin_1), J4.1 (Pin_1)
