File: Hardware/ParkerOnboardingProj/ParkerOnboardingProj.kicad_pcb (KiCad board)
At the start: 2 copper layers, 0 parts

Commit message: finished onboarding pcb
Parts:
- added D1: LED_PURPLE, layout:LED_0603_Symbol_on_F.SilkS, F.Cu at (47.0, 40.0)
- added J1: Conn_01x02, Connector_Molex:Molex_KK-254_AE-6410-02A_1x02_P2.54mm_Vertical, F.Cu at (42.0, 40.8)
- added R1: 105, Resistor_SMD:R_0603_1608Metric_Pad0.98x0.95mm_HandSolder, F.Cu at (47.4, 37.5)
- added REF**: MountingHole_3.2mm_M3, MountingHole:MountingHole_3.2mm_M3, F.Cu at (40.5, 33.0)
- added REF**: MountingHole_3.2mm_M3, MountingHole:MountingHole_3.2mm_M3, F.Cu at (52.0, 40.5)
- added SW1: SW_Push, Button_Switch_SMD:SW_DIP_SPSTx01_Slide_6.7x4.1mm_W6.73mm_P2.54mm_LowProfile_JPin, F.Cu at (49.0, 34.0)
Routing:
- net Net-(R1-Pad1): track 0.00 -> 7.69 mm
- net +3V3: track 0.00 -> 5.73 mm
- net GND: track 0.00 -> 2.83 mm, vias 0 -> 1
- net Net-(D1-A): track 0.00 -> 2.72 mm
- added copper zone on F.Cu, net +3V3
- added copper zone on B.Cu, net GND
Other:
- board outline added: 18.5 x 14.5 mm
