File: Hardware/akhily2_Horns_v1.0/akhily2_Horns_v1.0.kicad_sch (KiCad schematic)
At the start: 0 parts

Commit message: Completed Horns Board schematic, passes ERC
Parts:
- added C1, C2, C3: 0.1uF, symbol Device:C_Polarized
- added C4, C5: 1uF, symbol Device:C_Polarized
- added C6, C7: 10uF, symbol Device:C_Polarized
- added C8: 100uF, symbol Device:C_Polarized
- added C9: 0.1uF, symbol device:C
- added D1: ES2DA-13-F, symbol Device:D
- added F1: 2A, symbol device:Fuse
- added J1: Conn_01x03, symbol Connector_Generic:Conn_01x03
- added J2, J3, J4: Conn_01x02, symbol Connector_Generic:Conn_01x02
- added Q1: Q_NMOS_GSD, symbol device:Q_NMOS_GSD
- added R1: 1k, symbol Device:R
Connections:
- new net: J3.2 (Pin_2), J4.1 (Pin_1)
- new net: F1.2, Q1.3 (D)
- new net +24V: C1.1, C2.1, C3.1, C4.1, C5.1, C6.1, C7.1, C8.1, D1.1 (K), J1.2 (Pin_2), J3.1 (Pin_1)
- new net GND: C1.2, C2.2, C3.2, C4.2, C5.2, C6.2, C7.2, C8.2, C9.2, J1.1 (Pin_1), J1.3 (Pin_3), J2.2 (Pin_2), Q1.2 (S), R1.2
- new net HORN_CTL: C9.1, J2.1 (Pin_1), Q1.1 (G), R1.1
- new net HORN_IN: D1.2 (A), F1.1, J4.2 (Pin_2)

Commit message: Updated title block with name, title, revision 1.0
Other:
- title: Template -> Horns Board Schematic
Changed lines of the file:
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@@
 	(paper "USLetter")
 	(title_block
-		(title "Template")
+		(title "Horns Board Schematic")
 		(date "2022-08-16")
-		(rev "0.0")
+		(rev "1.0")
 		(company "Illini Solar Car")
-		(comment 1 "Designed By: Your Name")
+		(comment 1 "Designed By: Akhil Yerrapally")
 	)
 	(junction

Commit message: Save work before applying fixes
Parts:
- C1, C2, C3, C4, C5, C6, C7, C8, C9: footprint (none) -> Capacitor_THT:CP_Radial_D5.0mm_P2.00mm
- D1: footprint (none) -> Diode_THT:D_DO-41_SOD81_P10.16mm_Horizontal
- F1: footprint (none) -> Fuse:Fuseholder_Cylinder-5x20mm_Schurter_FAB_0031-355x_Horizontal_Closed
- J1: footprint (none) -> Connector_PinHeader_2.54mm:PinHeader_1x03_P2.54mm_Vertical
- J2, J3, J4: footprint (none) -> Connector_PinHeader_2.54mm:PinHeader_1x02_P2.54mm_Vertical
- Q1: footprint (none) -> Package_TO_SOT_SMD:TO-252-2
- R1: footprint (none) -> Resistor_THT:R_Axial_DIN0207_L6.3mm_D2.5mm_P10.16mm_Horizontal
Changed lines of the file:
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@@
 			)
 		)
-		(property "Footprint" ""
+		(property "Footprint" "Capacitor_THT:CP_Radial_D5.0mm_P2.00mm"
 			(at 130.5052 49.53 0)
 			(effects
@@
 			)
 		)
-		(property "Footprint" ""
+		(property "Footprint" "Capacitor_THT:CP_Radial_D5.0mm_P2.00mm"
 			(at 53.0352 134.62 0)
 			(effects
@@
 			)
 		)
-		(property "Footprint" ""
+		(property "Footprint" "Resistor_THT:R_Axial_DIN0207_L6.3mm_D2.5mm_P10.16mm_Horizontal"
 			(at 118.872 45.72 90)
 			(effects
@@
 			)
 		)
-		(property "Footprint" ""
+		(property "Footprint" "Connector_PinHeader_2.54mm:PinHeader_1x02_P2.54mm_Vertical"
 			(at 99.06 33.02 0)
 			(effects
@@
 			)
 		)
-		(property "Footprint" ""
+		(property "Footprint" "Fuse:Fuseholder_Cylinder-5x20mm_Schurter_FAB_0031-355x_Horizontal_Closed"
 			(at 108.712 66.04 90)
 			(effects
@@
 			)
 		)
-		(property "Footprint" ""
+		(property "Footprint" "Capacitor_THT:CP_Radial_D5.0mm_P2.00mm"
 			(at 32.7152 102.87 0)
 			(effects
@@
 			)
 		)
-		(property "Footprint" ""
+		(property "Footprint" "Capacitor_THT:CP_Radial_D5.0mm_P2.00mm"
 			(at 73.3552 102.87 0)
 			(effects
@@
 			)
 		)
-		(property "Footprint" ""
+		(property "Footprint" "Connector_PinHeader_2.54mm:PinHeader_1x03_P2.54mm_Vertical"
 			(at 69.85 44.45 0)
 			(effects
@@
 			)
 		)
-		(property "Footprint" ""
+		(property "Footprint" "Package_TO_SOT_SMD:TO-252-2"
 			(at 113.03 73.66 0)
 			(effects
@@
 			)
 		)
-		(property "Footprint" ""
+		(property "Footprint" "Capacitor_THT:CP_Radial_D5.0mm_P2.00mm"
 			(at 32.7152 133.35 0)
 			(effects
@@
 			)
 		)
-		(property "Footprint" ""
+		(property "Footprint" "Capacitor_THT:CP_Radial_D5.0mm_P2.00mm"
 			(at 93.6752 102.87 0)
 			(effects
@@
 			)
 		)
-		(property "Footprint" ""
+		(property "Footprint" "Diode_THT:D_DO-41_SOD81_P10.16mm_Horizontal"
 			(at 121.92 104.14 0)
 			(effects
@@
 			)
 		)
-		(property "Footprint" ""
+		(property "Footprint" "Connector_PinHeader_2.54mm:PinHeader_1x02_P2.54mm_Vertical"
 			(at 80.01 59.69 0)
 			(effects
@@
 			)
 		)
-		(property "Footprint" ""
+		(property "Footprint" "Connector_PinHeader_2.54mm:PinHeader_1x02_P2.54mm_Vertical"
 			(at 99.06 44.45 0)
 			(effects
@@
 			)
 		)
-		(property "Footprint" ""
+		(property "Footprint" "Capacitor_THT:CP_Radial_D5.0mm_P2.00mm"
 			(at 73.3552 134.62 0)
 			(effects
@@
 			)
 		)
-		(property "Footprint" ""
+		(property "Footprint" "Capacitor_THT:CP_Radial_D5.0mm_P2.00mm"
 			(at 93.6752 134.62 0)
 			(effects
@@
 			)
 		)
-		(property "Footprint" ""
+		(property "Footprint" "Capacitor_THT:CP_Radial_D5.0mm_P2.00mm"
 			(at 53.0352 102.87 0)
 			(effects

Commit message: Horns board specs, schematic, layout, gerbers
Parts:
- added D2: LED_GREEN, LED_SMD:LED_0805_2012Metric, symbol Device:LED
- added R2: 10k, Resistor_SMD:R_0805_2012Metric, symbol Device:R
- added TP1: +24V, TestPoint:TestPoint_Pad_D2.0mm, symbol Connector:TestPoint
- added TP2: GND, TestPoint:TestPoint_Pad_D2.0mm, symbol Connector:TestPoint
- added TP3: HORN_CTL, TestPoint:TestPoint_Pad_D2.0mm, symbol Connector:TestPoint
- added TP4: HORN_IN, TestPoint:TestPoint_Pad_D2.0mm, symbol Connector:TestPoint
- C1, C2, C3: value 0.1uF -> 0.1uF 50V; footprint Capacitor_THT:CP_Radial_D5.0mm_P2.00mm -> Capacitor_SMD:C_0805_2012Metric; symbol Device:C_Polarized -> device:C
- C4, C5: value 1uF -> 1uF 50V; footprint Capacitor_THT:CP_Radial_D5.0mm_P2.00mm -> Capacitor_SMD:C_0805_2012Metric; symbol Device:C_Polarized -> device:C
- C6, C7: value 10uF -> 10uF 50V; footprint Capacitor_THT:CP_Radial_D5.0mm_P2.00mm -> Capacitor_SMD:C_1206_3216Metric; symbol Device:C_Polarized -> device:C
- C8: value 100uF -> 100uF 50V; footprint Capacitor_THT:CP_Radial_D5.0mm_P2.00mm -> Capacitor_THT:CP_Radial_D8.0mm_P3.50mm
- C9: value 0.1uF -> 0.1uF 50V; footprint Capacitor_THT:CP_Radial_D5.0mm_P2.00mm -> Capacitor_SMD:C_0805_2012Metric
- D1: footprint Diode_THT:D_DO-41_SOD81_P10.16mm_Horizontal -> Diode_SMD:D_SMA
- F1: footprint Fuse:Fuseholder_Cylinder-5x20mm_Schurter_FAB_0031-355x_Horizontal_Closed -> Fuse:Fuse_1206_3216Metric
- Q1: value Q_NMOS_GSD -> IRFR010PBF; symbol device:Q_NMOS_GSD -> device:Q_NMOS_GDS
- R1: footprint Resistor_THT:R_Axial_DIN0207_L6.3mm_D2.5mm_P10.16mm_Horizontal -> Resistor_SMD:R_0805_2012Metric
Connections:
- net +24V: now also R2.1, TP1.1
- net GND: now also Q1.3 (S), D2.1 (K), TP2.1; no longer Q1.2 (S)
- net HORN_CTL: now also TP3.1
- net HORN_IN: now also TP4.1
- net HORN_MID: now reaches J3.2 (Pin_2), J4.1 (Pin_1)
- net at F1.2: now also Q1.2 (D); no longer Q1.3 (D)
- new net: D2.2 (A), R2.2
Other:
- note added: "Power indicator"
- note added: "Test points"
