File: Hardware/abfern_Horns_v1.0/abfernhorns.kicad_pcb (KiCad board)
At the start: 2 copper layers, 0 parts

Commit message: added gerber files
Parts:
- added C1: .1uF, Capacitor_SMD:C_0603_1608Metric_Pad1.08x0.95mm_HandSolder, F.Cu at (93.5, 70.9)
- added C2: .1u, Capacitor_SMD:C_0603_1608Metric_Pad1.08x0.95mm_HandSolder, F.Cu at (93.4, 74.7)
- added C3: .1u, Capacitor_SMD:C_0603_1608Metric_Pad1.08x0.95mm_HandSolder, F.Cu at (93.4, 77.7)
- added C4: .1u, Capacitor_SMD:C_0603_1608Metric_Pad1.08x0.95mm_HandSolder, F.Cu at (93.4, 80.5)
- added C5: 1u, Capacitor_SMD:C_0603_1608Metric_Pad1.08x0.95mm_HandSolder, F.Cu at (93.3, 83.6)
- added C6: 1u, Capacitor_SMD:C_0603_1608Metric_Pad1.08x0.95mm_HandSolder, F.Cu at (93.4, 86.1)
- added C7: 10u, Capacitor_SMD:C_0603_1608Metric_Pad1.08x0.95mm_HandSolder, F.Cu at (93.4, 89.4)
- added C8: 10u, Capacitor_SMD:C_0603_1608Metric_Pad1.08x0.95mm_HandSolder, F.Cu at (95.7, 93.2)
- added C9: 100u, Capacitor_SMD:CP_Elec_3x5.3, F.Cu at (112.3, 69.0)
- added D2: Diode, Diode_SMD:D_SMA, F.Cu at (113.0, 92.2)
- added F1: 2A, Fuse:Fuse_0402_1005Metric_Pad0.77x0.64mm_HandSolder, F.Cu at (115.3, 87.5)
- added J1: PWR, Connector_Molex:Molex_KK-254_AE-6410-03A_1x03_P2.54mm_Vertical, F.Cu at (100.7, 93.0)
- added J2: Connection CTRL, Connector_Molex:Molex_KK-254_AE-6410-02A_1x02_P2.54mm_Vertical, F.Cu at (101.7, 70.4)
- added J3: Connector A, Connector_Molex:Molex_KK-254_AE-6410-02A_1x02_P2.54mm_Vertical, F.Cu at (113.8, 74.7)
- added J4: Connector B, Connector_Molex:Molex_KK-254_AE-6410-02A_1x02_P2.54mm_Vertical, F.Cu at (114.1, 82.6)
- added Q2: MOSFET, Package_TO_SOT_SMD:SOT-23, F.Cu at (100.8, 84.0)
- added R1: 1k, Resistor_SMD:R_0603_1608Metric_Pad0.98x0.95mm_HandSolder, F.Cu at (100.8, 77.3)
Routing:
- net +24V: track 0.00 -> 85.2 mm
- net GND: track 0.00 -> 70.6 mm
- net /Horn In: track 0.00 -> 19.8 mm
- net Net-(Q2-S): track 0.00 -> 17.2 mm
- net Net-(J3-Pin_1): track 0.00 -> 9.10 mm
- net /Horn Control: track 0.00 -> 7.55 mm
- net Net-(Q2-G): track 0.00 -> 7.08 mm
- net Net-(J4-Pin_1): track 0.00 -> 5.57 mm
Other:
- board outline added: 30.5 x 30.5 mm
