File: Hardware/abfern_Horns_v1.0/abfernhorns.kicad_sch (KiCad schematic)
At the start: 16 parts, among them J1 Conn_01x03_Male, J2 Connection CTRL, J4 Conn_01x02_Male, Q1 NMOSFET

Commit message: added gerber files
Parts:
- removed C2, C3, C4: 0.1u, symbol Device:C_Polarized
- removed C5, C6: 1u, symbol Device:C_Polarized
- removed C7, C8: 10u, symbol Device:C_Polarized
- removed D1: 1N4001, Diode_THT:D_DO-41_SOD81_P10.16mm_Horizontal, symbol Diode:1N4001
- removed Q1: NMOSFET, symbol ICs:IRF7503TRPBF
- added C2, C3, C4: .1u, Capacitor_SMD:C_0603_1608Metric_Pad1.08x0.95mm_HandSolder, symbol Device:C
- added C5, C6: 1u, Capacitor_SMD:C_0603_1608Metric_Pad1.08x0.95mm_HandSolder, symbol Device:C
- added C7, C8: 10u, Capacitor_SMD:C_0603_1608Metric_Pad1.08x0.95mm_HandSolder, symbol Device:C
- added D2: Diode, Diode_SMD:D_SMA, symbol Diode:US2DA
- added J3: Connector A, Connector_Molex:Molex_KK-254_AE-6410-02A_1x02_P2.54mm_Vertical, symbol Connector:Conn_01x02_Male
- added Q2: MOSFET, Package_TO_SOT_SMD:SOT-23, symbol Transistor_FET:AO3400A
- C1: footprint (none) -> Capacitor_SMD:C_0603_1608Metric_Pad1.08x0.95mm_HandSolder
- C9: footprint (none) -> Capacitor_SMD:CP_Elec_3x5.3
- F1: footprint (none) -> Fuse:Fuse_0402_1005Metric_Pad0.77x0.64mm_HandSolder
- J1: footprint (none) -> Connector_Molex:Molex_KK-254_AE-6410-03A_1x03_P2.54mm_Vertical
- J2: footprint (none) -> Connector_Molex:Molex_KK-254_AE-6410-02A_1x02_P2.54mm_Vertical; MPN (none) -> 22272021; Notes (none) -> https://www.molex.com/content/dam/molex/molex-dot-com/produ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
- J4: value Conn_01x02_Male -> Connector B; footprint (none) -> Connector_Molex:Molex_KK-254_AE-6410-02A_1x02_P2.54mm_Vertical; MPN (none) -> 22272021; Notes (none) -> https://www.molex.com/content/dam/molex/molex-dot-com/produ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
- R1: footprint (none) -> Resistor_SMD:R_0603_1608Metric_Pad0.98x0.95mm_HandSolder
Connections:
- net +24V: now also C2.1, C3.1, C4.1, C5.1, C6.1, C7.1, C8.1, D2.1 (K), J3.2 (Pin_2)
- net GND: now also C2.2, C3.2, C4.2, C5.2, C6.2, C7.2, C8.2
- net Horn In: now also D2.2 (A), Q2.3 (D)
- net at C1.1: now also Q2.2 (S)
- net at R1.2: now also Q2.1 (G)
- net at J4.2 (Pin_2): now also J3.1 (Pin_1)
