File: Hardware/Proj_1/Template_v0.0.kicad_sch (KiCad schematic)
At the start: 4 parts, among them J1 Conn_01x02, SW1 SW_Push

Commit message: Proj_1 Hardware Complete
Parts:
- removed D1: LED_RED, layout:LED_0603_Symbol_on_F.SilkS, symbol Device:LED
- removed R1: 105, Resistor_SMD:R_0201_0603Metric_Pad0.64x0.40mm_HandSolder, symbol Device:R
- added D1: LED_RED, layout:LED_0603_Symbol_on_F.SilkS, symbol device:LED
- added R1: 105, Resistor_SMD:R_0603_1608Metric_Pad0.98x0.95mm_HandSolder, symbol device:R_US
- J1: MPN (none) -> 022272021
- SW1: MPN 1825910-6 -> 1825910-6; notes https://www.te.com/commerce/DocumentDelivery/DDEController?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 -> (none)
Connections:
- net GND: now also D1.1 (K)
- net at SW1.2: now also R1.1
- new net: D1.2 (A), R1.2
Other:
- title: Project 1, Hardware -> LED Project
