File: Hardware/Proj_1/_restore_backup_2026-09-25T03-00-51-409/Template_v0.0.kicad_sch (KiCad schematic)
At the start: 4 parts, among them J1 Conn_01x02, SW1 SW_Push

Commit message: Proj_1 Hardware Complete
Parts:
- removed D1: LED, layout:LED_0603_Symbol_on_F.SilkS, symbol Device:LED
- removed R1: 105, Resistor_SMD:R_0603_1608Metric_Pad0.98x0.95mm_HandSolder, symbol Device:R
- added D1: LED_RED, layout:LED_0603_Symbol_on_F.SilkS, symbol device:LED
- added R1: 105, Resistor_SMD:R_0603_1608Metric_Pad0.98x0.95mm_HandSolder, symbol device:R_US
Connections:
- net GND: now also D1.1 (K)
- net at SW1.2: now also R1.1
- net +3.3VA renamed +3V3
- new net: D1.2 (A), R1.2
