File: Hardware/jacobtk5_Horns_v1.0/jacobtk5_Horns_v1.0.kicad_pcb (KiCad board)
At the start: 2 copper layers, 0 parts

Commit message: Completed horn board layout
Parts:
- added C1: 0.1uF, Capacitor_SMD:CP_Elec_3x5.3, F.Cu at (160.5, 94.1)
- added C2: .1uF, Capacitor_SMD:CP_Elec_3x5.3, F.Cu at (130.2, 106.2)
- added C3: .1uF, Capacitor_SMD:CP_Elec_3x5.3, F.Cu at (130.2, 111.0)
- added C4: .1uF, Capacitor_SMD:CP_Elec_3x5.3, F.Cu at (137.0, 101.3)
- added C5: 1uF, Capacitor_SMD:CP_Elec_3x5.3, F.Cu at (137.0, 106.2)
- added C6: 1uF, Capacitor_SMD:CP_Elec_3x5.3, F.Cu at (137.0, 111.0)
- added C7: 10uF, Capacitor_SMD:CP_Elec_3x5.3, F.Cu at (143.8, 101.3)
- added C8: 10uF, Capacitor_SMD:CP_Elec_3x5.3, F.Cu at (143.8, 106.2)
- added C9: 100uF, Capacitor_THT:CP_Radial_D8.0mm_P3.50mm, F.Cu at (143.3, 113.0)
- added D1: ES2DA-13-F, Diode_SMD:D_SMB, F.Cu at (152.0, 105.0)
- added F1: 2A, Fuse:Fuse_0402_1005Metric, F.Cu at (155.7, 102.0)
- added J1: Conn_01x03, Connector_Molex:Molex_KK-254_AE-6410-03A_1x03_P2.54mm_Vertical, F.Cu at (152.9, 111.4)
- added J2: Horn Control, Connector_Molex:Molex_KK-254_AE-6410-02A_1x02_P2.54mm_Vertical, F.Cu at (131.4, 95.4)
- added J3: Horn Out, Connector_Molex:Molex_KK-254_AE-6410-02A_1x02_P2.54mm_Vertical, F.Cu at (143.4, 95.4)
- added J4: Horn Out, Connector_Molex:Molex_KK-254_AE-6410-02A_1x02_P2.54mm_Vertical, F.Cu at (151.6, 95.4)
- added Q1: IRFR010PBF, Package_TO_SOT_SMD:TO-252-3_TabPin2, F.Cu at (163.4, 101.7)
- added R1: 1k, Resistor_SMD:R_0603_1608Metric_Pad0.98x0.95mm_HandSolder, F.Cu at (138.6, 90.3)
- added REF**: MountingHole_3.2mm_M3_Pad, MountingHole:MountingHole_3.2mm_M3_Pad, F.Cu at (165.9, 114.8)
- added REF**: MountingHole_3.2mm_M3_Pad, MountingHole:MountingHole_3.2mm_M3_Pad, F.Cu at (124.1, 114.9)
- added REF**: MountingHole_3.2mm_M3_Pad, MountingHole:MountingHole_3.2mm_M3_Pad, F.Cu at (165.6, 86.2)
- added REF**: MountingHole_3.2mm_M3_Pad, MountingHole:MountingHole_3.2mm_M3_Pad, F.Cu at (124.7, 86.2)
Routing:
- net GND: track 0.00 -> 79.6 mm, vias 0 -> 1
- net Net-(Q1-G): track 0.00 -> 26.5 mm
- net /Horn In: track 0.00 -> 10.5 mm
- net Net-(Q1-D): track 0.00 -> 9.45 mm
- net /Horn Control: track 0.00 -> 6.62 mm
- net Net-(J3-Pin_2): track 0.00 -> 5.72 mm
- added copper zone on F.Cu, net +24V
- added copper zone on B.Cu, net GND
Other:
- board outline added: 50 x 37 mm
