File: Hardware/jacobtk5_Horns_v1.0/jacobtk5_Horns_v1.0.kicad_sch (KiCad schematic)
At the start: 0 parts

Commit message: Completed horn board layout
Parts:
- added C1: 0.1uF, Capacitor_SMD:CP_Elec_3x5.3, symbol device:C
- added C2, C3, C4: .1uF, Capacitor_SMD:CP_Elec_3x5.3, symbol device:C
- added C5, C6: 1uF, Capacitor_SMD:CP_Elec_3x5.3, symbol device:C
- added C7, C8: 10uF, Capacitor_SMD:CP_Elec_3x5.3, symbol device:C
- added C9: 100uF, Capacitor_SMD:CP_Elec_3x5.3, symbol Device:C_Polarized_US
- added D1: ES2DA-13-F, Diode_SMD:D_SMB, symbol device:D
- added F1: 2A, Fuse:Fuse_0402_1005Metric, symbol Device:Fuse
- added J1: Conn_01x03, Connector_Molex:Molex_KK-254_AE-6410-03A_1x03_P2.54mm_Vertical, symbol Connector_Generic:Conn_01x03
- added J2: Horn Control, Connector_Molex:Molex_KK-254_AE-6410-02A_1x02_P2.54mm_Vertical, symbol Connector_Generic:Conn_01x02
- added J3, J4: Horn Out, Connector_Molex:Molex_KK-254_AE-6410-02A_1x02_P2.54mm_Vertical, symbol Connector_Generic:Conn_01x02
- added Q1: IRFR010PBF, Package_TO_SOT_SMD:TO-252-3_TabPin2, symbol device:Q_NMOS_GDS
- added R1: 1k, Resistor_SMD:R_0603_1608Metric_Pad0.98x0.95mm_HandSolder, symbol device:R_Small_US
Connections:
- new net: J3.2 (Pin_2), J4.1 (Pin_1)
- new net: C1.1, Q1.1 (G), R1.2
- new net: F1.1, Q1.2 (D)
- new net +24V: C2.1, C3.1, C4.1, C5.1, C6.1, C7.1, C8.1, C9.1, D1.1 (K), J1.2 (Pin_2), J3.1 (Pin_1)
- new net GND: C1.2, C2.2, C3.2, C4.2, C5.2, C6.2, C7.2, C8.2, C9.2, J1.1 (Pin_1), J1.3 (Pin_3), J2.1 (Pin_1), Q1.3 (S)
- new net Horn Control: J2.2 (Pin_2), R1.1
- new net Horn In: D1.2 (A), F1.2, J4.2 (Pin_2)

Commit message: Changed led to LED in Heartbeat firmware
Parts:
- C9: footprint Capacitor_SMD:CP_Elec_3x5.3 -> Capacitor_THT:CP_Radial_D8.0mm_P3.50mm
Changed lines of the file:
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@@
 			)
 		)
-		(property "Footprint" "Capacitor_SMD:CP_Elec_3x5.3"
+		(property "Footprint" "Capacitor_THT:CP_Radial_D8.0mm_P3.50mm"
 			(at 90.17 130.81 0)
 			(effects
