File: Hardware/coulson5_Horns_v1.0/coulson5_Horns_v1.0.kicad_sch (KiCad schematic)
At the start: 0 parts

Commit message: Firemware Project 1
Other:
- title: Template -> Horns_v1.0
Changed lines of the file:
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@@
-(kicad_sch (version 20211123) (generator eeschema)
-  (paper "USLetter")
-  (title_block
-    (title "Template")
-    (date "2022-08-16")
-    (rev "0.0")
-    (company "Illini Solar Car")
-    (comment 1 "Designed By: Your Name")
-  )
-  (sheet_instances
-    (path "/" (page "1"))
-  )
+(kicad_sch
+	(version 20250114)
+	(generator "eeschema")
+	(generator_version "9.0")
+	(paper "USLetter")
+	(title_block
+		(title "Horns_v1.0")
+		(date "2026-09-22")
+		(rev "0.0")
+		(company "Illini Solar Car")
+		(comment 1 "Designed By: Steven Coulson")
+	)
+	(sheet_instances
+		(path "/"
+			(page "1")
+		)
+	)
+	(embedded_fonts no)
 )
