File: Hardware/hardproject/hardproj.kicad_pcb (KiCad board)
At the start: 2 copper layers, 0 parts

Commit message: Completed hardproj PCB design
Parts:
- added C1: 0.1u, Capacitor_SMD:C_0603_1608Metric_Pad1.08x0.95mm_HandSolder, F.Cu at (135.1, 96.0)
- added C2: 0.1u, Capacitor_SMD:C_0603_1608Metric_Pad1.08x0.95mm_HandSolder, F.Cu at (124.1, 100.0)
- added C3: 0.1u, Capacitor_SMD:C_0603_1608Metric_Pad1.08x0.95mm_HandSolder, F.Cu at (124.1, 103.0)
- added C4: 0.1u, Capacitor_SMD:C_0603_1608Metric_Pad1.08x0.95mm_HandSolder, F.Cu at (124.1, 106.0)
- added C5: 1u, Capacitor_SMD:C_0603_1608Metric_Pad1.08x0.95mm_HandSolder, F.Cu at (124.1, 109.0)
- added C6: 1u, Capacitor_SMD:C_0603_1608Metric_Pad1.08x0.95mm_HandSolder, F.Cu at (124.1, 112.0)
- added C7: 10u, Capacitor_SMD:C_0603_1608Metric_Pad1.08x0.95mm_HandSolder, F.Cu at (128.1, 112.0)
- added C8: 10u, Capacitor_SMD:C_0603_1608Metric_Pad1.08x0.95mm_HandSolder, F.Cu at (132.1, 112.0)
- added C9: 100u, Capacitor_THT:C_Radial_D8.0mm_H11.5mm_P3.50mm, F.Cu at (148.2, 109.0)
- added D1: ES2DA-13-F, Diode_SMD:D_SMA, F.Cu at (150.0, 95.8)
- added F2: 2A, Fuse:Fuse_0603_1608Metric_Pad1.05x0.95mm_HandSolder, F.Cu at (150.1, 100.1)
- added J1: Conn_01x03, Connector_Molex:Molex_KK-254_AE-6410-03A_1x03_P2.54mm_Vertical, F.Cu at (136.9, 109.0)
- added J2: HornControl, Connector_Molex:Molex_KK-254_AE-6410-02A_1x02_P2.54mm_Vertical, F.Cu at (131.5, 101.0)
- added J3: HornOut1, Connector_Molex:Molex_KK-254_AE-6410-02A_1x02_P2.54mm_Vertical, F.Cu at (140.5, 89.0)
- added J4: HornOut2, Connector_Molex:Molex_KK-254_AE-6410-02A_1x02_P2.54mm_Vertical, F.Cu at (149.0, 89.0)
- added Q1: IRFR010PBF, Package_TO_SOT_SMD:TO-252-2, F.Cu at (128.6, 89.5)
- added R1: 1k, Resistor_SMD:R_0603_1608Metric_Pad0.98x0.95mm_HandSolder, F.Cu at (127.1, 96.0)
- added REF**: MountingHole_3.2mm_M3, MountingHole:MountingHole_3.2mm_M3, F.Cu at (159.0, 111.0)
- added REF**: MountingHole_3.2mm_M3, MountingHole:MountingHole_3.2mm_M3, F.Cu at (115.0, 88.4)
- added REF**: MountingHole_3.2mm_M3, MountingHole:MountingHole_3.2mm_M3, F.Cu at (159.0, 88.1)
- added REF**: MountingHole_3.2mm_M3, MountingHole:MountingHole_3.2mm_M3, F.Cu at (115.0, 111.0)
Routing:
- net GND: track 0.00 -> 63.8 mm, vias 0 -> 3
- net Net-(Q1-D): track 0.00 -> 27.4 mm
- net Net-(Q1-G): track 0.00 -> 25.6 mm
- net /HornIn: track 0.00 -> 22.1 mm
- net /HornCTL: track 0.00 -> 7.61 mm
- net Net-(J3-Pin_2): track 0.00 -> 6.00 mm
- added copper zone on F.Cu, net +24V
- added copper zone on B.Cu, net GND
Other:
- board outline added: 52 x 32 mm
