File: Hardware/rowanpw2_Horns_v1.0/Horns_v1.0.kicad_pcb (KiCad board)
At the start: 2 copper layers, 0 parts

Commit message: Horns v1.0: complete PCB layout and Gerbers
Parts:
- added C1: .1uF, Capacitor_SMD:C_0603_1608Metric_Pad1.08x0.95mm_HandSolder, F.Cu at (130.1, 84.0)
- added C2: .1uF, Capacitor_SMD:C_0603_1608Metric_Pad1.08x0.95mm_HandSolder, F.Cu at (130.1, 89.0)
- added C3: .1uF, Capacitor_SMD:C_0603_1608Metric_Pad1.08x0.95mm_HandSolder, F.Cu at (139.1, 88.0)
- added C4: .1uF, Capacitor_SMD:C_0603_1608Metric_Pad1.08x0.95mm_HandSolder, F.Cu at (135.1, 91.0)
- added C5: 1uF, Capacitor_SMD:C_0603_1608Metric_Pad1.08x0.95mm_HandSolder, F.Cu at (135.1, 97.0)
- added C6: 1uF, Capacitor_SMD:C_0603_1608Metric_Pad1.08x0.95mm_HandSolder, F.Cu at (140.1, 97.0)
- added C7: 10uF, Capacitor_SMD:C_0603_1608Metric_Pad1.08x0.95mm_HandSolder, F.Cu at (145.1, 97.0)
- added C8: 10uF, Capacitor_SMD:C_0603_1608Metric_Pad1.08x0.95mm_HandSolder, F.Cu at (150.9, 97.0)
- added C9: 100uF, Capacitor_SMD:CP_Elec_8x10, F.Cu at (138.0, 80.0)
- added D1: S2JTR, Diode_SMD:D_SMB, F.Cu at (160.2, 88.0)
- added F1: 2A, Fuse:Fuse_1206_3216Metric_Pad1.42x1.75mm_HandSolder, F.Cu at (137.0, 66.5)
- added F2: 2A, Fuse:Fuse_1206_3216Metric_Pad1.42x1.75mm_HandSolder, F.Cu at (134.0, 71.5)
- added J1: Conn_Power_Supply, Connector_Molex:Molex_KK-254_AE-6410-03A_1x03_P2.54mm_Vertical, F.Cu at (147.5, 80.0)
- added J2: Conn_Horn_Control, Connector_Molex:Molex_KK-254_AE-6410-02A_1x02_P2.54mm_Vertical, F.Cu at (143.5, 90.0)
- added J3: Horn_Out_2, Connector_Molex:Molex_KK-254_AE-6410-02A_1x02_P2.54mm_Vertical, F.Cu at (158.5, 79.0)
- added J4: Horn_Out_1, Connector_Molex:Molex_KK-254_AE-6410-02A_1x02_P2.54mm_Vertical, F.Cu at (153.5, 69.0)
- added Q1: Q_NMOS_GDS, Package_TO_SOT_SMD:TO-252-2, F.Cu at (144.2, 70.7)
- added R1: 1k, Resistor_SMD:R_0603_1608Metric_Pad0.98x0.95mm_HandSolder, F.Cu at (130.1, 79.0)
- added REF**: M1, MountingHole:MountingHole_3.2mm_M3, F.Cu at (163.0, 68.0)
- added REF**: M2, MountingHole:MountingHole_3.2mm_M3, F.Cu at (163.0, 97.0)
- added REF**: M4, MountingHole:MountingHole_3.2mm_M3, F.Cu at (129.0, 68.0)
- added REF**: M3, MountingHole:MountingHole_3.2mm_M3, F.Cu at (129.0, 97.0)
Routing:
- net +24V: track 0.00 -> 120.7 mm, vias 0 -> 4
- net GND: track 0.00 -> 87.5 mm
- net /Horn_In: track 0.00 -> 52.7 mm
- net /Horn_Ctl: track 0.00 -> 27.5 mm
- net Net-(Q1-G): track 0.00 -> 18.9 mm
- net Net-(Q1-S): track 0.00 -> 15.7 mm, vias 0 -> 2
- net Net-(J3-Pin_1): track 0.00 -> 12.6 mm
- net Net-(C1-Pad1): track 0.00 -> 5.71 mm
- added copper zone on F.Cu, net +24V
- added copper zone on B.Cu, net GND
Other:
- board outline added: 42 x 37 mm
