File: Hardware/agrimj3_Horns_v1.0/Horns_v1.0.kicad_pcb (KiCad board)
At the start: 2 copper layers, 0 parts

Commit message: Hardware Project 2 PCB layout
Parts:
- added C1: 0.1uF, Capacitor_SMD:C_0805_2012Metric, F.Cu at (135.5, 68.0)
- added C2: 1uF, Capacitor_SMD:C_0805_2012Metric, F.Cu at (135.2, 73.0)
- added C3: 0.1uF, Capacitor_SMD:C_0805_2012Metric, F.Cu at (135.1, 78.0)
- added C4: 0.1uF, Capacitor_SMD:C_0805_2012Metric, F.Cu at (139.5, 68.0)
- added C5: 1uF, Capacitor_SMD:C_0805_2012Metric, F.Cu at (139.6, 73.0)
- added C6: 100uF, Capacitor_SMD:C_0805_2012Metric, F.Cu at (139.6, 78.0)
- added C7: 10uF, Capacitor_SMD:C_0805_2012Metric, F.Cu at (143.9, 68.0)
- added C8: 0.1uF, Capacitor_SMD:C_0805_2012Metric, F.Cu at (144.1, 73.0)
- added C9: 10uF, Capacitor_SMD:C_0805_2012Metric, F.Cu at (143.9, 78.0)
- added D1: 1N4001, Diode_SMD:D_SMB, F.Cu at (137.8, 85.0)
- added F1: Fuse, Fuse:Fuse_1812_4532Metric, F.Cu at (145.5, 85.0)
- added J1: Conn_01x02, Connector_Molex:Molex_KK-254_AE-6410-02A_1x02_P2.54mm_Vertical, F.Cu at (152.5, 65.2)
- added J5: Conn_01x02, Connector_Molex:Molex_KK-254_AE-6410-02A_1x02_P2.54mm_Vertical, F.Cu at (127.0, 75.0)
- added J6: Conn_01x03, Connector_Molex:Molex_KK-254_AE-6410-03A_1x03_P2.54mm_Vertical, F.Cu at (134.0, 60.5)
- added J7: Conn_01x02, Connector_Molex:Molex_KK-254_AE-6410-02A_1x02_P2.54mm_Vertical, F.Cu at (152.5, 74.5)
- added Q1: Q_NMOS_GDS, Package_TO_SOT_SMD:TO-252-2, F.Cu at (126.5, 85.9)
- added R1: 1k, Resistor_SMD:R_0805_2012Metric, F.Cu at (130.5, 70.1)
- added REF**: MountingHole_3.7mm, MountingHole:MountingHole_3.7mm, F.Cu at (153.5, 89.0)
- added REF**: MountingHole_3.7mm, MountingHole:MountingHole_3.7mm, F.Cu at (124.5, 60.5)
Routing:
- net GND: track 0.00 -> 66.2 mm, vias 0 -> 1
- net /Horn In: track 0.00 -> 28.5 mm
- net /Horn Control: track 0.00 -> 16.9 mm
- net Net-(J7-Pin_2): track 0.00 -> 10.8 mm
- net Net-(J1-Pin_2): track 0.00 -> 6.74 mm
- net Net-(C1-Pad1): track 0.00 -> 5.36 mm
- net +24V: track 0.00 -> 1.54 mm
- added copper zone on F.Cu, net +24V
- added copper zone on B.Cu, net GND
Other:
- board outline added: 41.5 x 40.5 mm
