File: Hardware/agrimj3_Horns_v1.0/Horns_v1.0.kicad_sch (KiCad schematic)
At the start: 16 parts, among them J1 Conn_01x02_Male, J2 Conn_01x02_Female, J3 Conn_01x03_Male, J4 Conn_01x02_Female, Q2 Q_NMOS

Commit message: Hardware Project 2 PCB layout
Parts:
- removed J1: Conn_01x02_Male, symbol Connector:Conn_01x02_Male
- removed J2, J4: Conn_01x02_Female, symbol Connector:Conn_01x02_Female
- removed J3: Conn_01x03_Male, symbol Connector:Conn_01x03_Male
- removed Q2: Q_NMOS, symbol Device:Q_NMOS
- added D1: 1N4001, Diode_SMD:D_SMB, symbol Diode:1N4001
- added J1, J5, J7: Conn_01x02, Connector_Molex:Molex_KK-254_AE-6410-02A_1x02_P2.54mm_Vertical, symbol Connector_Generic:Conn_01x02
- added J6: Conn_01x03, Connector_Molex:Molex_KK-254_AE-6410-03A_1x03_P2.54mm_Vertical, symbol Connector_Generic:Conn_01x03
- added Q1: Q_NMOS_GDS, Package_TO_SOT_SMD:TO-252-2, symbol device:Q_NMOS_GDS
- C1, C2, C3, C4, C5, C6, C7, C8, C9: footprint (none) -> Capacitor_SMD:C_0805_2012Metric
- F1: footprint (none) -> Fuse:Fuse_1812_4532Metric
- R1: footprint (none) -> Resistor_SMD:R_0805_2012Metric
Connections:
- net +24V: now also D1.1 (K), J1.1 (Pin_1), J6.2 (Pin_2)
- net GND: now also J5.2 (Pin_2), J6.1 (Pin_1), J6.3 (Pin_3), Q1.2 (D)
- net Horn Control: now also J5.1 (Pin_1), Q1.1 (G)
- net Horn In: now also D1.2 (A), Q1.3 (S)
- net at F1.2: now also J7.2 (Pin_2)
- new net: J1.2 (Pin_2), J7.1 (Pin_1)
