File: Hardware/ckeng2_Horns_v1.0/Horns_Board.kicad_pcb (KiCad board)
At the start: 2 copper layers, 0 parts

Commit message: Finish PCB layout design, deleted the unnecessary fuse 1. Both zones are GND to simplify GND Connection
Parts:
- added C1: 0.1u, Capacitor_SMD:C_0603_1608Metric_Pad1.08x0.95mm_HandSolder, F.Cu at (99.0, 99.0)
- added C2: 0.1u, Capacitor_SMD:C_0603_1608Metric_Pad1.08x0.95mm_HandSolder, F.Cu at (110.6, 106.8)
- added C3: 0.1u, Capacitor_SMD:C_0603_1608Metric_Pad1.08x0.95mm_HandSolder, F.Cu at (110.6, 105.0)
- added C4: 0.1u, Capacitor_SMD:C_0603_1608Metric_Pad1.08x0.95mm_HandSolder, F.Cu at (108.5, 109.5)
- added C5: 1u, Capacitor_SMD:C_0603_1608Metric_Pad1.08x0.95mm_HandSolder, F.Cu at (106.9, 105.8)
- added C6: 1u, Capacitor_SMD:C_0603_1608Metric_Pad1.08x0.95mm_HandSolder, F.Cu at (106.9, 107.5)
- added C7: 10u, Capacitor_SMD:C_0603_1608Metric_Pad1.08x0.95mm_HandSolder, F.Cu at (103.1, 107.5)
- added C8: 10u, Capacitor_SMD:C_0603_1608Metric_Pad1.08x0.95mm_HandSolder, F.Cu at (103.1, 105.8)
- added C9: 100u, Capacitor_SMD:CP_Elec_6.3x5.3, F.Cu at (106.0, 101.0)
- added D1: D, Diode_SMD:D_SMB, F.Cu at (102.8, 111.8)
- added D2: LED_RED, layout:LED_0603_Symbol_on_F.SilkS, F.Cu at (100.0, 103.7)
- added F2: 2A, Fuse:Fuse_0603_1608Metric_Pad1.05x0.95mm_HandSolder, F.Cu at (108.9, 113.2)
- added J1: Power Ins, Connector_Molex:Molex_KK-254_AE-6410-03A_1x03_P2.54mm_Vertical, F.Cu at (107.5, 93.5)
- added J2: Horn Ctl Ins, Connector_Molex:Molex_KK-254_AE-6410-02A_1x02_P2.54mm_Vertical, F.Cu at (94.0, 102.0)
- added J3: Horn Outs, Connector_Molex:Molex_KK-254_AE-6410-02A_1x02_P2.54mm_Vertical, F.Cu at (115.0, 102.0)
- added J4: Horn Outs, Connector_Molex:Molex_KK-254_AE-6410-02A_1x02_P2.54mm_Vertical, F.Cu at (115.0, 112.3)
- added Q1: Q_NMOS_GDS, Package_TO_SOT_SMD:TO-252-2, F.Cu at (104.7, 118.0)
- added R1: 1K, Resistor_SMD:R_0603_1608Metric_Pad0.98x0.95mm_HandSolder, F.Cu at (99.5, 107.5)
- added REF**: MountingHole_3.2mm_M3, MountingHole:MountingHole_3.2mm_M3, F.Cu at (115.0, 93.5)
- added REF**: MountingHole_3.2mm_M3, MountingHole:MountingHole_3.2mm_M3, F.Cu at (94.0, 118.5)
- added REF**: MountingHole_3.2mm_M3, MountingHole:MountingHole_3.2mm_M3, F.Cu at (94.0, 93.5)
- added REF**: MountingHole_3.2mm_M3, MountingHole:MountingHole_3.2mm_M3, F.Cu at (115.0, 118.5)
Routing:
- net +24V: track 0.00 -> 50.9 mm
- net /HORN_CTL: track 0.00 -> 27.5 mm
- net /HORN_IN: track 0.00 -> 14.4 mm
- net Net-(J3-Pin_1): track 0.00 -> 7.73 mm
- net Net-(Q1-D): track 0.00 -> 6.02 mm
- net Net-(D2-K): track 0.00 -> 2.29 mm
- net GND: vias 0 -> 2
- added copper zone on B.Cu, net GND
- added copper zone on F.Cu, net GND
Other:
- board outline added: 29 x 34 mm
