File: Hardware/proj2/proj2_kicad_v0.0.kicad_pcb (KiCad board)
At the start: 2 copper layers, 45 x 29 mm, 22 parts, among them J1 Conn_01x03, Q1(MOSFET_SW?)1 DMN2058U

Commit message: push containing my greenlit Horns project
Parts:
- moved C5 1.90 mm to (128.8, 106.4)
- moved C7 1.85 mm to (133.6, 106.2)
- moved C6 1.00 mm to (135.0, 102.0), turned to -90 degrees
- moved C4 0.96 mm to (130.0, 102.0), turned to -90 degrees
Routing:
- net GND: track 29.7 -> 23.1 mm, vias 3 -> 4
- net /Horn In: track 35.0 -> 33.1 mm
- net +24V: track 17.2 -> 18.2 mm
- net Net-(Q1(MOSFET_SW?)1-D): track 7.61 -> 6.89 mm
