File: Hardware/rwproj1/rwproj1.kicad_pcb (KiCad board)
At the start: 2 copper layers, 0 parts

Commit message: HW P1
Parts:
- added D1: LED_RED, layout:LED_0603_Symbol_on_F.SilkS, F.Cu at (133.2, 100.0)
- added J1: Conn_01x02, Connector_Molex:Molex_KK-254_AE-6410-02A_1x02_P2.54mm_Vertical, F.Cu at (133.5, 106.0)
- added R1: 105Ω, Resistor_SMD:R_0603_1608Metric_Pad0.98x0.95mm_HandSolder, F.Cu at (137.1, 100.0)
- added REF**: MountingHole_3.2mm_M3, MountingHole:MountingHole_3.2mm_M3, F.Cu at (134.0, 94.0)
- added REF**: MountingHole_3.2mm_M3, MountingHole:MountingHole_3.2mm_M3, F.Cu at (142.0, 107.0)
- added SW1: SW_Push, Button_Switch_SMD:SW_DIP_SPSTx01_Slide_6.7x4.1mm_W8.61mm_P2.54mm_LowProfile, F.Cu at (142.0, 95.7)
Routing:
- net Net-(R1-Pad1): track 0.00 -> 11.1 mm
- net GND: track 0.00 -> 2.58 mm, vias 0 -> 1
- net Net-(D1-A): track 0.00 -> 2.18 mm
- added copper zone on F.Cu, net +3V3
- added copper zone on B.Cu, net GND
Other:
- board outline added: 16 x 22 mm
