File: Hardware/aaabra_Horns_v1.0/aaabra_Horns_v1.0.kicad_sch (KiCad schematic)
At the start: 0 parts

Commit message: Horns schematic complete
Parts:
- added C1, C2, C3, C4: .1u, symbol device:C
- added C5, C6: 1u, symbol device:C
- added C7, C8: 10u, symbol device:C
- added C9: 100u, symbol Device:C_Polarized
- added D1: ES2DA, symbol Device:D
- added F1: 2, symbol Device:Fuse
- added J1: Conn_01x03, symbol Connector_Generic:Conn_01x03
- added J2, J3, J4: Conn_01x02, symbol Connector_Generic:Conn_01x02
- added Q1: IRFR010PBF, symbol device:Q_NMOS_GDS
- added R1: 1k, symbol Device:R
Connections:
- new net: F1.2, J3.1 (Pin_1)
- new net: J3.2 (Pin_2), J4.1 (Pin_1)
- new net +24V: C2.1, C3.1, C4.1, C5.1, C6.1, C7.1, C8.1, C9.1, D1.1 (K), F1.1, J1.2 (Pin_2)
- new net GND: C1.2, C2.2, C3.2, C4.2, C5.2, C6.2, C7.2, C8.2, C9.2, J1.1 (Pin_1), J1.3 (Pin_3), J2.1 (Pin_1), Q1.3 (S), R1.2
- new net HORN_CTL: C1.1, J2.2 (Pin_2), Q1.1 (G), R1.1
- new net Horn_In: D1.2 (A), J4.2 (Pin_2), Q1.2 (D)

Commit message: Refurnished Horns Schematic complete
Parts:
- C1, C2, C3, C4, C5, C6, C7, C8: footprint (none) -> Capacitor_SMD:C_0805_2012Metric
- C9: footprint (none) -> Capacitor_THT:CP_Radial_D5.0mm_P2.00mm
- D1: footprint (none) -> Diode_SMD:D_SMA
- F1: footprint (none) -> Fuse:Fuse_1206_3216Metric_Pad1.42x1.75mm_HandSolder
- J1: footprint (none) -> Connector_Molex:Molex_KK-254_AE-6410-03A_1x03_P2.54mm_Vertical
- J2, J3, J4: footprint (none) -> Connector_Molex:Molex_KK-254_AE-6410-02A_1x02_P2.54mm_Vertical
- Q1: footprint (none) -> Package_TO_SOT_SMD:TO-252-2
- R1: footprint (none) -> Resistor_SMD:R_0603_1608Metric_Pad0.98x0.95mm_HandSolder
Changed lines of the file:
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@@
 			)
 		)
-		(property "Footprint" ""
+		(property "Footprint" "Connector_Molex:Molex_KK-254_AE-6410-02A_1x02_P2.54mm_Vertical"
 			(at 87.63 97.79 0)
 			(effects
@@
 			)
 		)
-		(property "Footprint" ""
+		(property "Footprint" "Capacitor_SMD:C_0805_2012Metric"
 			(at 107.6452 149.86 0)
 			(effects
@@
 			)
 		)
-		(property "Footprint" ""
+		(property "Footprint" "Capacitor_SMD:C_0805_2012Metric"
 			(at 138.1252 149.86 0)
 			(effects
@@
 			)
 		)
-		(property "Footprint" ""
+		(property "Footprint" "Resistor_SMD:R_0603_1608Metric_Pad0.98x0.95mm_HandSolder"
 			(at 88.392 115.57 90)
 			(effects
@@
 			)
 		)
-		(property "Footprint" ""
+		(property "Footprint" "Fuse:Fuse_1206_3216Metric_Pad1.42x1.75mm_HandSolder"
 			(at 96.52 90.678 90)
 			(effects
@@
 			)
 		)
-		(property "Footprint" ""
+		(property "Footprint" "Capacitor_SMD:C_0805_2012Metric"
 			(at 117.8052 149.86 0)
 			(effects
@@
 			)
 		)
-		(property "Footprint" ""
+		(property "Footprint" "Package_TO_SOT_SMD:TO-252-2"
 			(at 106.68 104.14 0)
 			(effects
@@
 			)
 		)
-		(property "Footprint" ""
+		(property "Footprint" "Connector_Molex:Molex_KK-254_AE-6410-03A_1x03_P2.54mm_Vertical"
 			(at 138.43 102.87 0)
 			(effects
@@
 			)
 		)
-		(property "Footprint" ""
+		(property "Footprint" "Capacitor_THT:CP_Radial_D5.0mm_P2.00mm"
 			(at 148.2852 149.86 0)
 			(effects
@@
 			)
 		)
-		(property "Footprint" ""
+		(property "Footprint" "Capacitor_SMD:C_0805_2012Metric"
 			(at 97.4852 149.86 0)
 			(effects
@@
 			)
 		)
-		(property "Footprint" ""
+		(property "Footprint" "Connector_Molex:Molex_KK-254_AE-6410-02A_1x02_P2.54mm_Vertical"
 			(at 110.49 96.52 0)
 			(effects
@@
 			)
 		)
-		(property "Footprint" ""
+		(property "Footprint" "Capacitor_SMD:C_0805_2012Metric"
 			(at 87.3252 149.86 0)
 			(effects
@@
 			)
 		)
-		(property "Footprint" ""
+		(property "Footprint" "Capacitor_SMD:C_0805_2012Metric"
 			(at 127.9652 149.86 0)
 			(effects
@@
 			)
 		)
-		(property "Footprint" ""
+		(property "Footprint" "Capacitor_SMD:C_0805_2012Metric"
 			(at 100.0252 119.38 0)
 			(effects
@@
 			)
 		)
-		(property "Footprint" ""
+		(property "Footprint" "Capacitor_SMD:C_0805_2012Metric"
 			(at 77.1652 149.86 0)
 			(effects
@@
 			)
 		)
-		(property "Footprint" ""
+		(property "Footprint" "Connector_Molex:Molex_KK-254_AE-6410-02A_1x02_P2.54mm_Vertical"
 			(at 110.49 88.9 0)
 			(effects
@@
 			)
 		)
-		(property "Footprint" ""
+		(property "Footprint" "Diode_SMD:D_SMA"
 			(at 114.3 106.68 0)
 			(effects

Commit message: Horns board schematic
Other:
- title: Template -> Horns Board Schematic
Changed lines of the file:
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@@
 	(paper "USLetter")
 	(title_block
-		(title "Template")
-		(date "2022-08-16")
+		(title "Horns Board Schematic")
+		(date "2026-09-24")
 		(rev "0.0")
 		(company "Illini Solar Car")
-		(comment 1 "Designed By: Your Name")
+		(comment 1 "Designed By: Andrew Abraham")
 	)
 	(junction

Commit message: onboarding
Connections:
- net +24V: now also F1.2; no longer F1.1
- net at J3.1 (Pin_1): now also F1.1; no longer F1.2
Other:
- moved on the sheet: C1, D1, F1, J1, J2, J3, J4, R1
