File: Hardware/HProject-OB_HARD/HPROJECT-OB_HARD.kicad_sch (KiCad schematic)
At the start: 17 parts, among them J1 PWR, J2 Hrn_Ctrl, J3 Hrn_Out1, J4 Hrn_Out2, M1 MPMOS

Commit message: onboarding project fixes
Parts:
- R2: value R -> 1K ohm
Connections:
- net +24V: now also C6.2; no longer C6.1
- net GND: now also C6.1; no longer C6.2
Other:
- moved on the sheet: C6

Commit message: Glingle Onboarding Projects - updated
Parts:
- removed M1: MPMOS, Connector_Molex:Molex_KK-254_AE-6410-04A_1x04_P2.54mm_Vertical, symbol pspice:MPMOS
- added Q1: IRF740, Package_TO_SOT_THT:TO-220-3_Vertical, symbol Transistor_FET:IRF740
- C1, C10, C2, C3: footprint Capacitor_SMD:CP_Elec_3x5.3 -> Capacitor_SMD:C_0402_1005Metric_Pad0.74x0.62mm_HandSolder
- C4, C5: footprint Capacitor_SMD:CP_Elec_4x3 -> Capacitor_SMD:C_0402_1005Metric
- C6, C7: footprint Capacitor_SMD:CP_Elec_4x5.3 -> Capacitor_SMD:C_0603_1608Metric_Pad1.08x0.95mm_HandSolder
- C8: footprint Capacitor_SMD:CP_Elec_6.3x5.4 -> Capacitor_THT:CP_Radial_D6.3mm_P2.50mm
- J1: footprint Connector_Molex:Molex_CLIK-Mate_502382-0270_1x02-1MP_P1.25mm_Vertical -> Connector_Molex:Molex_KK-254_AE-6410-03A_1x03_P2.54mm_Vertical
- R2: footprint Connector_Molex:Molex_KK-254_AE-6410-02A_1x02_P2.54mm_Vertical -> Resistor_THT:R_Axial_DIN0207_L6.3mm_D2.5mm_P10.16mm_Horizontal
Connections:
- net GND: now also F1.1, J1.1 (Pin_1), J1.3 (Pin_3)
- net Horn In: now also Q1.2 (D)
- net HornSignal: now also Q1.1 (G)
- net at F1.2: now also Q1.3 (S)
